Commit message: Comenzando a adaptar el Rbwatcher a Ignition 6

File: Robotnik_ws/src/robot_description/urdf/wheels/rubber_wheel/rubber_wheel(antigua).urdf.xacro (robot description, xacro)
@@ -10,13 +10,13 @@
                                           mesh_file:=robot_description/meshes/wheels/rubber_wheel/rubber_wheel_right">
 <!--WHEEL TIRE -->
-    <joint name="${prefix}_wheel_joint" type="continuous">
+    <joint name="${robot_id}_wheel_joint" type="continuous">
       <parent link="${parent}"/>
-      <child link="${prefix}_wheel"/>
+      <child link="${robot_id}_wheel"/>
       <xacro:insert_block name="origin" />
       <axis xyz="0 1 0" rpy="0 0 0" />
       <limit effort="100" velocity="100"/>
-      <joint_properties damping="0.0" friction="0.0"/>
+      <joint_properties damping="0.5" friction="2.0"/>
     </joint>
-    <link name="${prefix}_wheel">
+    <link name="${robot_id}_wheel">
       <visual>
         <!-- HIGH RESOLUTION WHEELS -->
@@ -41,13 +41,8 @@
       </visual>
       <collision>
-          <xacro:unless value="${reflect}">
-            <origin xyz="0 0 0" rpy="0 0 0" />
-          </xacro:unless>
-          <xacro:if value="${reflect}">
-            <origin xyz="0 0 0" rpy="${M_PI} 0 0" />
-          </xacro:if>
+          <origin xyz="0 0 0" rpy="${M_PI/2} 0 0" />
           <geometry>
-						<mesh filename="package://${mesh_file}.stl" />
-        </geometry>
+						<cylinder length="${rubber_wheel_width}" radius="${rubber_wheel_radius}" />
+          </geometry>
       </collision>
       <inertial>
@@ -57,18 +52,11 @@
       </inertial>
     </link>
-    <!-- Transmission is important to link the joints and the controller (see summit_xl_control/config/summit_xl_control.yaml)-->
-    <transmission name="${prefix}_wheel_joint_trans">
-      <type>transmission_interface/SimpleTransmission</type>
-      <joint name="${prefix}_wheel_joint">
-        <hardwareInterface>hardware_interface/VelocityJointInterface</hardwareInterface>
-      </joint>
-      <actuator name="${prefix}_wheel_joint_motor">
-        <mechanicalReduction>1</mechanicalReduction>
-        <motorTorqueConstant>20</motorTorqueConstant>
-      </actuator>
-     </transmission>
-    <gazebo reference="${prefix}_wheel">
-			<material>Gazebo/Black</material>
-			<turnGravityOff>false</turnGravityOff>
+    <gazebo reference="${robot_id}_wheel">
+			<!-- <material>Gazebo/Black</material> -->
+      <mu1>0.9</mu1>
+      <mu2>0.5</mu2>
+      <kp>2.75e9</kp>
+      <kd>8.25e1</kd>
+      <fdir1>1 0 0</fdir1>
 		</gazebo>
   </xacro:macro>

File: Robotnik_ws/src/robotnik_sensors/robotnik_sensors/urdf/3d_lidar/robosense_helios_16p.urdf.xacro (robot description, xacro)
@@ -51,13 +51,7 @@
   </xacro:macro>
   <xacro:macro name="sensor_robosense_helios_16p_gazebo">
-      <xacro:if value="${gpu}">
-        <xacro:property name="ray_type" value="gpu_ray" />
-      </xacro:if>
-      <xacro:unless value="${gpu}">
-        <xacro:property name="ray_type" value="ray" />
-      </xacro:unless>
       <gazebo reference="${frame_prefix}link">
-        <sensor type="${ray_type}" name="${frame_prefix}sensor">
-          <pose>0 0 0 0 0 0</pose>
+        <sensor type="gpu_lidar" name="${frame_prefix}sensor">
+          <pose>0.0 0.0 0.0 0.0 0.0 0.0</pose>
           <visualize>false</visualize>
           <update_rate>10</update_rate>
@@ -78,25 +72,16 @@
             </scan>
             <range>
-              <min>0.10</min>
-              <max>50</max>
+              <min>0.05</min>
+              <max>100</max>
               <resolution>0.001</resolution>
             </range>
             <noise>
               <type>gaussian</type>
-              <mean>0.0</mean>
+              <mean>0.01</mean>
               <stddev>0.00</stddev>
             </noise>
           </ray>
-          <plugin name="${node_name}" filename="libgazebo_ros_velodyne_laser.so">
-            <ros>
-              <namespace>${node_namespace}</namespace>
-              <remapping>~/out:=${topic_prefix}point_cloud</remapping>
-            </ros>
-            <frame_name>${frame_prefix}link</frame_name>
-            <min_range>0.05</min_range>
-            <max_range>100.0</max_range>
-            <gaussian_noise>0.01</gaussian_noise>
-            <organize_cloud>0</organize_cloud>
-          </plugin>
+          <topic>${topic_prefix}/point_cloud</topic>
+          <ignition_frame_id>${frame_prefix}link</ignition_frame_id>
         </sensor>
       </gazebo>

File: Robotnik_ws/src/robotnik_sensors/robotnik_sensors/urdf/all_sensors.urdf.xacro (robot description, xacro)
@@ -43,3 +43,7 @@
   <xacro:include filename="$(find robotnik_sensors)/urdf/camera/axis_m5525.urdf.xacro" />
   <xacro:include filename="$(find robotnik_sensors)/urdf/camera/axis_m5526.urdf.xacro" />
+    <!-- BLK ARC -->
+  <xacro:include filename="$(find robotnik_sensors)/urdf/blk_arc.urdf.xacro" />
+    <!-- Link 750 -->
+  <xacro:include filename="$(find robotnik_sensors)/urdf/link_750_nh.urdf.xacro" />
 </robot>

File: Robotnik_ws/src/robotnik_sensors/robotnik_sensors/urdf/gps/ublox.urdf.xacro (robot description, xacro)
@@ -85,5 +85,7 @@
 			</vertical_sensing>
 			</gps>
-			<plugin name="${node_name}" filename="libgazebo_ros_gps_sensor.so">
+			<topic>${topic_prefix}</topic>
+          		<ignition_frame_id>${frame_prefix}link</ignition_frame_id>
+			<!--plugin name="${node_name}" filename="libgazebo_ros_gps_sensor.so">
 			<ros>
 				<namespace>${node_namespace}</namespace>
@@ -91,5 +93,5 @@
 				<remapping>~/vel:=${topic_prefix}vel</remapping>
 			</ros>
-			</plugin>
+			</plugin-->
 		</sensor>
 		</gazebo>
