Commit message: Arreglo de sensores de Rbwatcher
La mayoría de sensores se han arreglado, ahora bien, hay un problemas con las juntas prismáticas y revolutes por el que los TFs dan error, así que por ahora las he dejado como juntas fijas

File: Robotnik_ws/src/robot_description/robots/rbwatcher/rbwatcher.urdf.xacro (robot description, xacro)
@@ -73,5 +73,5 @@
         </xacro:sensor_ublox>
     	<!-- LIDAR -->
-    	<xacro:sensor_robosense_helios_16p frame_prefix="$(arg prefix)top_3d_laser" node_namespace="$(arg namespace)" topic_prefix="top_3d_laser" parent="$(arg prefix)base_link" gpu="$(arg gpu)" >
+    	<xacro:sensor_robosense_helios_16p frame_prefix="$(arg prefix)top_3d_laser" node_namespace="$(arg namespace)" topic_prefix="top_3d_laser" parent="$(arg prefix)base_link" gpu="$(arg gpu)" simulation="$(arg gazebo_classic)">
     	  	<origin xyz="-0.11924 0.0 0.38609" rpy="0 0 0"/>
     	</xacro:sensor_robosense_helios_16p>
@@ -93,5 +93,5 @@
 			</xacro:sensor_blk_arc>
 		</xacro:if>
-		<xacro:rbrobout_gz_ignition_control namespace="$(arg namespace)" prefix="$(arg prefix)"/>
+		<xacro:rbwatcher_gz_ignition_control namespace="$(arg namespace)" prefix="$(arg prefix)"/>
         	<xacro:ros_diff_move_gazebo_ignition_front prefix="$(arg prefix)"/>
         	<xacro:ros_diff_move_gazebo_ignition_rear prefix="$(arg prefix)"/>

File: Robotnik_ws/src/robot_description/simulators/gazebo_ignition/rbwatcher/rbwatcher_control.urdf.xacro (robot description, xacro)
@@ -1,5 +1,5 @@
 <?xml version="1.0"?>
 <robot xmlns:xacro="http://wiki.ros.org/xacro">
-    <xacro:macro name="rbrobout_gz_ignition_control"  params="namespace prefix">
+    <xacro:macro name="rbwatcher_gz_ignition_control"  params="namespace prefix">
         <gazebo>
           <plugin name="ign_ros2_control::IgnitionROS2ControlPlugin" filename="ign_ros2_control-system">
@@ -41,6 +41,6 @@
              <left_joint>${prefix}front_left_wheel_joint</left_joint>
 	     <right_joint>${prefix}front_right_wheel_joint</right_joint>
-             <wheel_separation>0.5</wheel_separation>
-             <wheel_radius>0.22</wheel_radius>
+             <wheel_separation>0.31</wheel_separation>
+             <wheel_radius>0.11</wheel_radius>
              <odom_publish_frequency>1</odom_publish_frequency>
              <topic>cmd_vel</topic>
@@ -58,6 +58,6 @@
 	     <left_joint>${prefix}back_left_wheel_joint</left_joint>
 	     <right_joint>${prefix}back_right_wheel_joint</right_joint>
-             <wheel_separation>0.573</wheel_separation>
-             <wheel_radius>0.127</wheel_radius>
+             <wheel_separation>0.31</wheel_separation>
+             <wheel_radius>0.11</wheel_radius>
              <odom_publish_frequency>0</odom_publish_frequency>
              <publish_odom>false</publish_odom>

File: Robotnik_ws/src/robotnik_sensors/robotnik_sensors/urdf/3d_lidar/robosense_helios_16p.urdf.xacro (robot description, xacro)
@@ -5,5 +5,5 @@
                        parent
                        *origin
-                       simulation:=false
+                       simulation:=true
                        node_name:=robosense_helios_16p
                        node_namespace:=${None}
@@ -72,6 +72,6 @@
             </scan>
             <range>
-              <min>0.05</min>
-              <max>100</max>
+              <min>0.2</min>
+              <max>50</max>
               <resolution>0.001</resolution>
             </range>

File: Robotnik_ws/src/robotnik_sensors/robotnik_sensors/urdf/link_750_nh.urdf (copia).xacro (robot description, xacro)
@@ -38,5 +38,5 @@
       </collision>
     </link>
-    <joint name="${prefix}_pan_joint" type="fixed">
+    <joint name="${prefix}_pan_joint" type="revolute">
       <axis xyz="0 0 1"/>
       <origin xyz="0.0 0.0 0.0318" rpy="0 0 0"/>
@@ -81,5 +81,5 @@
       </actuator>
     </transmission>
-    <joint name="${prefix}_tilt_joint" type="fixed">
+    <joint name="${prefix}_tilt_joint" type="revolute">
       <axis xyz="0 0 1"/>
       <origin xyz="0.0 0.0 0.102" rpy="${PI/2} 0 0"/>
@@ -123,5 +123,5 @@
       </actuator>
     </transmission>
-    <joint name="${prefix}_zoom_color_joint" type="fixed">
+    <joint name="${prefix}_zoom_color_joint" type="prismatic">
       <axis xyz="0 0 1"/>
       <origin xyz="0.0 0.0 0.0" rpy="0 0 0"/>
@@ -210,5 +210,5 @@
       </xacro:if>
     </link>
-    <joint name="${prefix}_zoom_thermal_joint" type="fixed">
+    <joint name="${prefix}_zoom_thermal_joint" type="prismatic">
       <axis xyz="0 0 1"/>
       <origin xyz="0.0 0.0 0.0" rpy="0 0 0"/>
