Commit message: Rbwatcher urdf fix
He actualizado los xacro de Rbwatcher para conseguir acercarme lo máximo al modelo del rbrobout. Además, para este último he añadido un modelo con ascensor.

También he descubierto los errores que tenía con rbwatcher al importar al PROTO (hay que cambiar los daes por stl)

File: Robotnik_ws/src/robot_description/urdf/bases/rbwatcher/rbwatcher_base.urdf.xacro (robot description, xacro)
@@ -1,115 +1,77 @@
 <?xml version="1.0"?>
-<robot name="summit_xl" xmlns:xacro="http://wiki.ros.org/xacro">
-	<xacro:include filename="$(find robot_description)/urdf/wheels/rubber_wheel/rubber_wheel.urdf.xacro" />
-	<xacro:include filename="$(find robot_description)/urdf/wheels/omni_wheel/omni_wheel.urdf.xacro" />
-	<xacro:macro name="rbwatcher_base" params="prefix publish_bf hq kinematics:=skid_4w">
-		<!-- Robot mechanical and motor parameters -->
-		<xacro:property name="PI" value="3.1415926535897931"/>
-		<!-- Wheel parameters -->
-		<xacro:property name="wheel_offset_x" value="0.22795" />    <!-- x,y,z in translation from base_link to the center of the wheel -->
-		<xacro:property name="wheel_offset_y" value="0.155" />
-		<xacro:property name="wheel_offset_z" value="0.0" />
-		<xacro:property name="docking_contact_offset_x" value="0.29378" />
-		<xacro:property name="docking_contact_offset_y" value="0.0" />
-		<xacro:property name="docking_contact_offset_z" value="0.07321" />
-		<xacro:property name="rubber_wheel_radius" value="0.1175" />
-		<xacro:property name="rubber_wheel_width" value="0.142" />
-		<xacro:property name="rubber_wheel_mass" value="4" />
-		<xacro:property name="mesh_file_left" value="robot_description/meshes/wheels/rubber_wheel/rubber_wheel_v2_left" />
-		<xacro:property name="mesh_file_right" value="robot_description/meshes/wheels/rubber_wheel/rubber_wheel_v2_right" />
-		<!-- BASE FOOTPRINT -->
-		<xacro:if value="${publish_bf}">
-		<link name="${prefix}base_footprint">
-			<visual>
-				<origin xyz="0 0 0" rpy="0 0 0" />
-				<geometry>
-					<box size="0.001 0.001 0.001" />
-				</geometry>
-			</visual>
-		</link>
-		<joint name="${prefix}base_footprint_joint" type="fixed">
-			<origin xyz="0 0 ${rubber_wheel_radius}" rpy="0 0 0" /> <!-- ${wheel_radius} property must be defined inside wheel description -->
-			<parent link="${prefix}base_footprint"/>
-			<child link="${prefix}base_link" />
-		</joint>
-		</xacro:if>
-		<!-- BASE_LINK -->
-		<link name="${prefix}base_link">
-		<inertial>
-			<mass value="50.0" />
-			<origin xyz="0 0 0" />
-			<inertia  ixx="1.391" ixy="0.004"  ixz="0.0"  iyy="6.853"  iyz="0.0"  izz="6.125" />
-		</inertial>
-		<visual>
-			<origin xyz="0 0 0" rpy="0 0 0" />
-			<xacro:if value="${hq}">
-			<geometry>
-				<mesh filename="package://robot_description/meshes/bases/rbwatcher/rbwatcher_body.dae"/>
-			</geometry>
-			</xacro:if>
-			<xacro:unless value="${hq}">
-			<geometry>
-				<mesh filename="package://robot_description/meshes/bases/rbwatcher/rbwatcher_body.dae"/>
-			</geometry>
-			</xacro:unless>
-			<material name="darkgrey">
-				<color rgba="0.1 0.1 0.1 1"/>
-			</material>
-		</visual>
-		<collision>
-			<origin xyz="0 0 0" rpy="0 0 0 " />
-			<geometry>
-				<mesh filename="package://robot_description/meshes/bases/rbwatcher/rbwatcher_body.stl"/>
-			</geometry>
-		</collision>
-		</link>
-		<gazebo reference="${prefix}base_link">
-			<material>Gazebo/Gray</material>
-			<turnGravityOff>false</turnGravityOff>
-		</gazebo>
-		<!-- DOCKING CONTACTS -->
-		<joint name="${prefix}base_docking_joint" type="fixed">
-			<origin xyz="${docking_contact_offset_x} ${docking_contact_offset_y} ${docking_contact_offset_z}" rpy="0 0 0 " />
-			<parent link="${prefix}base_link"/>
-			<child link="${prefix}base_docking_contact_link" />
-		</joint>
-		<!-- DOCKING LINK -->
-		<link name="${prefix}base_docking_contact_link" />
-		<xacro:if value="${kinematics == 'skid' or kinematics == 'skid_4w'}">
-			<xacro:rubber_wheel prefix="${prefix}front_right" parent="${prefix}base_link" reflect="false" hq="${hq}" rubber_wheel_radius="${rubber_wheel_radius}"
-								rubber_wheel_width="${rubber_wheel_width}" rubber_wheel_mass="${rubber_wheel_mass}"
-								mesh_file="${mesh_file_right}">
-				<origin xyz="${wheel_offset_x} -${wheel_offset_y} ${wheel_offset_z}" rpy="0 0 0"/>
-			</xacro:rubber_wheel>
-			<xacro:rubber_wheel prefix="${prefix}front_left" parent="${prefix}base_link" reflect="false" hq="${hq}" rubber_wheel_radius="${rubber_wheel_radius}"
-								rubber_wheel_width="${rubber_wheel_width}" rubber_wheel_mass="${rubber_wheel_mass}"
-								mesh_file="${mesh_file_left}">
-				<origin xyz="${wheel_offset_x} ${wheel_offset_y} ${wheel_offset_z}" rpy="0 0 0"/>
-			</xacro:rubber_wheel>
-			<xacro:rubber_wheel prefix="${prefix}back_left" parent="${prefix}base_link" reflect="false" hq="${hq}" rubber_wheel_radius="${rubber_wheel_radius}"
-								rubber_wheel_width="${rubber_wheel_width}" rubber_wheel_mass="${rubber_wheel_mass}"
-								mesh_file="${mesh_file_left}">
-				<origin xyz="-${wheel_offset_x} ${wheel_offset_y} ${wheel_offset_z}" rpy="0 0 0"/>
-			</xacro:rubber_wheel>
-			<xacro:rubber_wheel prefix="${prefix}back_right" parent="${prefix}base_link" reflect="false" hq="${hq}" rubber_wheel_radius="${rubber_wheel_radius}"
-								rubber_wheel_width="${rubber_wheel_width}" rubber_wheel_mass="${rubber_wheel_mass}"
-								mesh_file="${mesh_file_right}">
-				<origin xyz="-${wheel_offset_x} -${wheel_offset_y} ${wheel_offset_z}" rpy="0 0 0"/>
-			</xacro:rubber_wheel>
-		</xacro:if>
-		<xacro:if value="${kinematics == 'omni' or kinematics == 'omni_4w'}">
-			<xacro:omni_wheel prefix="${prefix}front_right" parent="${prefix}base_link" reflect="false" hq="${hq}">
-				<origin xyz="${wheel_offset_x} -${wheel_offset_y} ${wheel_offset_z}" rpy="0 0 0"/>
-			</xacro:omni_wheel>
-			<xacro:omni_wheel prefix="${prefix}front_left" parent="${prefix}base_link" reflect="true" hq="${hq}">
-				<origin xyz="${wheel_offset_x} ${wheel_offset_y} ${wheel_offset_z}" rpy="0 0 0"/>
-			</xacro:omni_wheel>
-			<xacro:omni_wheel prefix="${prefix}back_left" parent="${prefix}base_link" reflect="true" hq="${hq}">
-				<origin xyz="-${wheel_offset_x} ${wheel_offset_y} ${wheel_offset_z}" rpy="0 0 0"/>
-			</xacro:omni_wheel>
-			<xacro:omni_wheel prefix="${prefix}back_right" parent="${prefix}base_link" reflect="false" hq="${hq}">
-				<origin xyz="-${wheel_offset_x} -${wheel_offset_y} ${wheel_offset_z}" rpy="0 0 0"/>
-			</xacro:omni_wheel>
-    	</xacro:if>
-	</xacro:macro>
+<robot name="rbwatcher" xmlns:xacro="http://wiki.ros.org/xacro">
+	<!-- ***************** -->
+	<!-- Imported elements -->
+	<!-- ***************** -->
+	<!-- First we import all posible elements defined in the urdf.xacro files. All these elements are defined as macro:xacros -->
+	<!-- Import RB-Watcher base elements -->
+	<xacro:include filename="$(find robot_description)/urdf/bodies/rbwatcher/rbwatcher_body.urdf.xacro" />
+	<!-- Import RB-Watcher wheels -->
+  	<xacro:include filename="$(find robot_description)/urdf/wheels/rubber_wheel/rubber_wheel.urdf.xacro" />
+  	<xacro:include filename="$(find robot_description)/urdf/wheels/omni_wheel/omni_wheel.urdf.xacro" />
+	<!-- Import all available sensors -->
+	<xacro:include filename="$(find robotnik_sensors)/urdf/all_sensors.urdf.xacro" />
+	<xacro:property name="PI" value="3.1415926535897931"/>
+	<!-- Wheel parameters -->
+	<xacro:property name="wheel_offset_x" value="0.22795" />    <!-- x,y,z in translation from base_link to the center of the wheel -->
+	<xacro:property name="wheel_offset_y" value="0.155" />
+	<xacro:property name="wheel_offset_z" value="0.0" />
+	<xacro:property name="docking_contact_offset_x" value="0.29378" />
+	<xacro:property name="docking_contact_offset_y" value="0.0" />
+	<xacro:property name="docking_contact_offset_z" value="0.07321" />
+	<xacro:property name="rubber_wheel_radius" value="0.1175" />
+	<xacro:property name="rubber_wheel_width" value="0.142" />
+	<xacro:property name="rubber_wheel_mass" value="4" />
+	<xacro:property name="mesh_file_left" value="robot_description/meshes/wheels/rubber_wheel/rubber_wheel_v2_left" />
+	<xacro:property name="mesh_file_right" value="robot_description/meshes/wheels/rubber_wheel/rubber_wheel_v2_right" />
+	<!-- Flag to select the high or low quality model -->
+	<xacro:property name="hq" value="true" />
+  <xacro:macro name="rbwatcher" params="prefix:=robot_ hq publish_bf">
+		<!-- *************** -->
+		<!-- Robots Elements -->
+		<!-- *************** -->
+		<!-- Here we create the robot elements using the xacro:macros imported at the beggining of this file -->
+		<xacro:rbwatcher_body prefix="${prefix}" />
+		<!-- Wheels -->
+		<xacro:rubber_wheel
+	            prefix="${prefix}front_right"
+	            parent="${prefix}base_link"
+	            reflect="false" hq="${hq}"
+	            rubber_wheel_radius="${rubber_wheel_radius}"
+	            rubber_wheel_width="${rubber_wheel_width}"
+	            rubber_wheel_mass="${rubber_wheel_mass}"
+		    mesh_file="${mesh_file_right}">
+		    <origin xyz="${wheel_offset_x} -${wheel_offset_y} ${wheel_offset_z}" rpy="0 0 0"/>
+		</xacro:rubber_wheel>
+		<xacro:rubber_wheel
+	            prefix="${prefix}front_left"
+	            parent="${prefix}base_link"
+	            reflect="false" hq="${hq}"
+	            rubber_wheel_radius="${rubber_wheel_radius}"
+	            rubber_wheel_width="${rubber_wheel_width}"
+	            rubber_wheel_mass="${rubber_wheel_mass}"
+		    mesh_file="${mesh_file_left}">
+		    <origin xyz="${wheel_offset_x} ${wheel_offset_y} ${wheel_offset_z}" rpy="0 0 0"/>
+		</xacro:rubber_wheel>
+		<xacro:rubber_wheel
+	            prefix="${prefix}back_right"
+	            parent="${prefix}base_link"
+	            reflect="false" hq="${hq}"
+	            rubber_wheel_radius="${rubber_wheel_radius}"
+	            rubber_wheel_width="${rubber_wheel_width}"
+	            rubber_wheel_mass="${rubber_wheel_mass}"
+		    mesh_file="${mesh_file_right}">
+		    <origin xyz="-${wheel_offset_x} -${wheel_offset_y} ${wheel_offset_z}" rpy="0 0 0"/>
+		</xacro:rubber_wheel>
+		<xacro:rubber_wheel
+	            prefix="${prefix}back_left"
+	            parent="${prefix}base_link"
+	            reflect="false" hq="${hq}"
+	            rubber_wheel_radius="${rubber_wheel_radius}"
+	            rubber_wheel_width="${rubber_wheel_width}"
+	            rubber_wheel_mass="${rubber_wheel_mass}"
+		    mesh_file="${mesh_file_left}">
+		    <origin xyz="-${wheel_offset_x} ${wheel_offset_y} ${wheel_offset_z}" rpy="0 0 0"/>
+		</xacro:rubber_wheel>
+   </xacro:macro>
 </robot>

File: Robotnik_ws/src/robot_description/urdf/bodies/rbwatcher/rbwatcher_body_sindae.urdf.xacro (robot description, xacro)
@@ -30,10 +30,10 @@
 		<xacro:if value="${hq}">
 		<geometry>
-			<mesh filename="package://robot_description/meshes/bases/rbwatcher/rbwatcher_body.dae"/>
+			<mesh filename="package://robot_description/meshes/bases/rbwatcher/rbwatcher_body.stl"/>
 		</geometry>
 		</xacro:if>
 		<xacro:unless value="${hq}">
 		<geometry>
-			<mesh filename="package://robot_description/meshes/bases/rbwatcher/rbwatcher_body.dae"/>
+			<mesh filename="package://robot_description/meshes/bases/rbwatcher/rbwatcher_body.stl"/>
 		</geometry>
 		</xacro:unless>

File: Robotnik_ws/src/robotnik_sensors/robotnik_sensors/urdf/3d_lidar/robosense_helios_16p.urdf.xacro (robot description, xacro)
@@ -1,9 +1,11 @@
 <?xml version="1.0"?>
 <robot name="sensor_robosense_helios" xmlns:xacro="http://wiki.ros.org/xacro">
+  <xacro:include filename="$(find robotnik_sensors)/urdf/3d_lidar/lidar_3d_plugin.urdf.xacro" />
   <xacro:macro name="sensor_robosense_helios_16p"
                params="frame_prefix
                        parent
                        *origin
-                       simulation:=true
+                       gazebo_classic:=false
+                       gazebo_ignition:=false
                        node_name:=robosense_helios_16p
                        node_namespace:=${None}
@@ -46,44 +48,18 @@
     </joint>
     <link name="${frame_prefix}link"/>
-    <xacro:if value="${simulation}">
-      <xacro:sensor_robosense_helios_16p_gazebo/>
-    </xacro:if>
-  </xacro:macro>
-  <xacro:macro name="sensor_robosense_helios_16p_gazebo">
-      <gazebo reference="${frame_prefix}link">
-        <sensor type="gpu_lidar" name="${frame_prefix}sensor">
-          <pose>0.0 0.0 0.0 0.0 0.0 0.0</pose>
-          <visualize>false</visualize>
-          <update_rate>10</update_rate>
-          <ray>
-            <scan>
-              <horizontal>
-                <samples>1200</samples>
-                <resolution>1.0</resolution>
-                <min_angle>${-radians(180)}</min_angle>
-                <max_angle>${radians(180)}</max_angle>
-              </horizontal>
-              <vertical>
-                <samples>32</samples>
-                <resolution>1.0</resolution>
-                <min_angle>0.0</min_angle>
-                <max_angle>${radians(85)}</max_angle>
-              </vertical>
-            </scan>
-            <range>
-              <min>0.2</min>
-              <max>50</max>
-              <resolution>0.001</resolution>
-            </range>
-            <noise>
-              <type>gaussian</type>
-              <mean>0.01</mean>
-              <stddev>0.00</stddev>
-            </noise>
-          </ray>
-          <topic>${topic_prefix}/point_cloud</topic>
-          <ignition_frame_id>${frame_prefix}link</ignition_frame_id>
-        </sensor>
-      </gazebo>
+    <xacro:lidar_3d_plugin
+      node_namespace="${node_namespace}"
+      node_name="${node_name}"
+      gazebo_classic="${gazebo_classic}"
+      gazebo_ignition="${gazebo_ignition}"
+      min_range="0.3"
+      max_range="100.0"
+      max_angle="85"
+      frame_link="${frame_prefix}link"
+      rate="10"
+      horizontal_samples="1200"
+      vertical_samples="16"
+    >
+    </xacro:lidar_3d_plugin>
   </xacro:macro>
 </robot>

File: Robotnik_ws/src/robotnik_sensors/robotnik_sensors/urdf/gps/ublox.urdf.xacro (robot description, xacro)
@@ -1,9 +1,11 @@
 <?xml version="1.0"?>
 <robot name="sensor_ublox" xmlns:xacro="http://wiki.ros.org/xacro">
+  <xacro:include filename="$(find robotnik_sensors)/urdf/gps/gps_plugin.urdf.xacro" />
 	<xacro:macro name="sensor_ublox"
 				params="frame_prefix
 						parent
 						*origin
-						simulation:=false
+						gazebo_classic:=false
+						gazebo_ignition:=false
 						node_name:=ublox
 						node_namespace:=${None}
@@ -50,51 +52,14 @@
 	    <gravity>true</gravity>
 	  </gazebo>
-    <xacro:if value="${simulation}">
-		<gazebo reference="${frame_prefix}base_link">
-		<sensor type="gps" name="${frame_prefix}sensor">
-			<always_on>true</always_on>
-			<update_rate>${update_rate}</update_rate>
-			<gps>
-			<position_sensing>
-				<horizontal>
-				<noise type="gaussian">
-					<mean>0.0</mean>
-					<stddev>0.1</stddev>
-				</noise>
-				</horizontal>
-				<vertical>
-				<noise type="gaussian">
-					<mean>0.0</mean>
-					<stddev>0.1</stddev>
-				</noise>
-				</vertical>
-			</position_sensing>
-			<vertical_sensing>
-				<horizontal>
-				<noise type="gaussian">
-					<mean>0.0</mean>
-					<stddev>0.1</stddev>
-				</noise>
-				</horizontal>
-				<vertical>
-				<noise type="gaussian">
-					<mean>0.0</mean>
-					<stddev>0.1</stddev>
-				</noise>
-				</vertical>
-			</vertical_sensing>
-			</gps>
-			<topic>${topic_prefix}</topic>
-          		<ignition_frame_id>${frame_prefix}link</ignition_frame_id>
-			<!--plugin name="${node_name}" filename="libgazebo_ros_gps_sensor.so">
-			<ros>
-				<namespace>${node_namespace}</namespace>
-				<remapping>~/out:=${topic_prefix}fix</remapping>
-				<remapping>~/vel:=${topic_prefix}vel</remapping>
-			</ros>
-			</plugin-->
-		</sensor>
-		</gazebo>
-    </xacro:if>
+    <xacro:gps_plugin
+      node_namespace="${node_namespace}"
+      node_name="${node_name}"
+      gazebo_classic="${gazebo_classic}"
+      gazebo_ignition="${gazebo_ignition}"
+      topic_prefix="${topic_prefix}_gps"
+      frame_link="${frame_prefix}base_link"
+      rate="${update_rate}"
+    >
+    </xacro:gps_plugin>
   </xacro:macro>
 </robot>
