Commit message: rbwatcher terminado en webots
La simulación del RbWatcher en webots se ha completado correctamente. Todos sus sensores y movimiento funciona.

File: Robotnik_ws/src/robot_description/urdf/bodies/rbwatcher/rbwatcher_body_condae.urdf.xacro (robot description, xacro)
@@ -30,10 +30,10 @@
 		<xacro:if value="${hq}">
 		<geometry>
-			<mesh filename="package://robot_description/meshes/bases/rbwatcher/rbwatcher_body.stl"/>
+			<mesh filename="package://robot_description/meshes/bases/rbwatcher/rbwatcher_body.dae"/>
 		</geometry>
 		</xacro:if>
 		<xacro:unless value="${hq}">
 		<geometry>
-			<mesh filename="package://robot_description/meshes/bases/rbwatcher/rbwatcher_body.stl"/>
+			<mesh filename="package://robot_description/meshes/bases/rbwatcher/rbwatcher_body.dae"/>
 		</geometry>
 		</xacro:unless>

File: Robotnik_ws/src/robot_description/urdf/structures/sensor_support/antena_std.urdf.xacro (robot description, xacro)
@@ -15,5 +15,5 @@
 	      <origin rpy="0 0 0" xyz="0 0 0"/>
 	      <geometry>
-	        <mesh filename="package://${mesh_file}.dae"/>
+	        <mesh filename="package://${mesh_file}.stl"/>
 	      </geometry>
 	    </visual>

File: Robotnik_ws/src/robot_description/urdf/structures/summit_hm/summit_hm_structure.xacro (robot description, xacro)
@@ -21,5 +21,5 @@
         </material>
 	      <geometry>
-	        <mesh filename="package://${mesh_file}.dae"/>
+	        <mesh filename="package://${mesh_file}.stl"/>
 	      </geometry>
 	    </visual>

File: Robotnik_ws/src/robot_description/urdf/wheels/rubber_wheel/rubber_wheel.urdf.xacro (robot description, xacro)
@@ -29,5 +29,5 @@
           </xacro:if>
           <geometry>
-							<mesh filename="package://${mesh_file}.dae" />
+							<mesh filename="package://${mesh_file}.stl" />
           </geometry>
         </xacro:if>
