Commit message: Nuevo mapa para simulaciones y otras cosas

File: Robotnik_ws/src/robot_description/robots/rbvogui/rbvogui.urdf.xacro (robot description, xacro)
@@ -5,28 +5,70 @@
     <!-- Imported elements -->
     <!-- ***************** -->
-    <!-- First we import all posible elements defined in the urdf.xacro files. All these elements are defined as macro:xacros -->
+    <!-- First we import all posible elements defined in the urdf.xacro files. All these elements
+    are defined as macro:xacros -->
     <!-- Import rbvogui base elements-->
-    <xacro:include filename="$(find robot_description)/urdf/bases/rbvogui/rbvogui_base.urdf.xacro" />
+    <xacro:include
+        filename="$(find robot_description)/urdf/bases/rbvogui/rbvogui_base.urdf.xacro" />
     <xacro:include filename="$(find robot_description)/urdf/base_hw/rbvogui.ros2_control.urdf" />
-    <xacro:include filename="$(find robot_description)/simulators/gazebo_classic/rbvogui/rbvogui_control.urdf.xacro" />
+    <xacro:include
+        filename="$(find robot_description)/simulators/gazebo_classic/rbvogui/rbvogui_control.urdf.xacro" />
+    <xacro:include
+        filename="$(find robot_description)/simulators/gazebo_ignition/rbvogui/rbvogui_control.urdf.xacro" />
     <!-- Import all available sensors -->
     <xacro:include filename="$(find robotnik_sensors)/urdf/all_sensors.urdf.xacro" />
-    <xacro:include filename="$(find robot_description)/urdf/structures/sensor_support/gps_mast.urdf.xacro" />
     <!-- Flag to select the high or low quality model -->
     <xacro:property name="hq" value="true" />
+    <xacro:property name="front_laser_offset_x" value="0.53" />
+    <xacro:property name="front_laser_offset_y" value="0.33" />
+    <xacro:property name="front_laser_offset_z" value="0.1145" />
+    <xacro:property name="rear_laser_offset_x" value="-0.53" />
+    <xacro:property name="rear_laser_offset_y" value="-0.33" />
+    <xacro:property name="rear_laser_offset_z" value="0.1145" />
+    <xacro:property name="imu_offset_x" value="0.127" />
+    <xacro:property name="imu_offset_y" value="-0.129" />
+    <xacro:property name="imu_offset_z" value="0.212" />
+    <xacro:property name="front_rgbd_camera_offset_x" value="0.46462" />
+    <xacro:property name="front_rgbd_camera_offset_y" value="0.0" />
+    <xacro:property name="front_rgbd_camera_offset_z" value="0.18258" />
+    <xacro:property name="rear_rgbd_camera_offset_x" value="-0.515" />
+    <xacro:property name="rear_rgbd_camera_offset_y" value="0.0" />
+    <xacro:property name="rear_rgbd_camera_offset_z" value="0.29" />
     <!-- Launch Arguments -->
-	<xacro:arg name="namespace" default="robot"/>
-	<xacro:arg name="prefix" default="robot_"/>
-	<xacro:arg name="gazebo_classic" default="false"/>
-    <xacro:rbvogui prefix="$(arg prefix)" hq="${hq}"/>
+    <xacro:arg name="namespace" default="robot" />
+    <xacro:arg name="prefix" default="robot_" />
+    <xacro:arg name="gazebo_classic" default="false" />
+    <xacro:arg name="gazebo_ignition" default="false" />
+    <xacro:rbvogui prefix="$(arg prefix)" hq="${hq}" />
     <!-- SENSORS see robotnik_sensors for the specific configuration -->
     <!-- IMU -->
     <xacro:sensor_vectornav
         frame_prefix="$(arg prefix)vectornav_"
-        parent="$(arg prefix)chassis_link"
+        parent="$(arg prefix)base_link"
         node_namespace="$(arg namespace)"
-        simulation="$(arg gazebo_classic)">
-        <origin xyz="0.3 -0.3 0.0725" rpy="0 0 0"/>
+        gazebo_classic="$(arg gazebo_classic)"
+        gazebo_ignition="$(arg gazebo_ignition)">
+        <origin xyz="${imu_offset_x} ${imu_offset_y} ${imu_offset_z}" rpy="0 0 0" />
     </xacro:sensor_vectornav>
+    <!-- LASERS -->
+    <xacro:sensor_sick_s300
+        frame_prefix="$(arg prefix)front_laser_"
+        parent="$(arg prefix)base_link"
+        node_namespace="$(arg namespace)"
+        node_name="front_laser"
+        gazebo_classic="$(arg gazebo_classic)"
+        gazebo_ignition="$(arg gazebo_ignition)">
+        <origin xyz="${front_laser_offset_x} ${front_laser_offset_y} ${front_laser_offset_z}"
+            rpy="0 ${-PI} ${-3/4*PI}" />
+    </xacro:sensor_sick_s300>
+    <xacro:sensor_sick_s300
+        frame_prefix="$(arg prefix)rear_laser_"
+        parent="$(arg prefix)base_link"
+        node_namespace="$(arg namespace)"
+        node_name="rear_laser"
+        gazebo_classic="$(arg gazebo_classic)"
+        gazebo_ignition="$(arg gazebo_ignition)">
+        <origin xyz="${rear_laser_offset_x} ${rear_laser_offset_y} ${rear_laser_offset_z}"
+            rpy="0 ${-PI} ${1/4*PI}" />
+    </xacro:sensor_sick_s300>
     <!-- Front Camera -->
     <xacro:sensor_intel_realsense_d435
@@ -35,40 +77,34 @@
         node_namespace="$(arg namespace)"
         node_name="front_camera"
-        simulation="$(arg gazebo_classic)">
-        <origin xyz="0.46462 0.0 0.18258" rpy="0 0 0"/>
+        gazebo_classic="$(arg gazebo_classic)"
+        gazebo_ignition="$(arg gazebo_ignition)">
+        <origin
+            xyz="${front_rgbd_camera_offset_x} ${front_rgbd_camera_offset_y} ${front_rgbd_camera_offset_z}"
+            rpy="0 0 0" />
     </xacro:sensor_intel_realsense_d435>
     <!-- Rear Camera -->
-    <!-- <xacro:sensor_intel_realsense_d435
+    <xacro:sensor_intel_realsense_d435
         frame_prefix="$(arg prefix)rear_rgbd_camera_"
-        parent="$(arg prefix)chassis_link"
+        parent="$(arg prefix)base_link"
         node_namespace="$(arg namespace)"
         node_name="rear_camera"
-        simulation="$(arg gazebo_classic)">
-        <origin xyz="-0.503 0.0 0.29" rpy="0 0 -${PI}"/>
-    </xacro:sensor_intel_realsense_d435> -->
-    <!-- 2d laser -->
-    <xacro:sensor_sick_s300
-        frame_prefix="$(arg prefix)front_laser_"
-        parent="$(arg prefix)chassis_link"
-        node_namespace="$(arg namespace)"
-        node_name="front_laser"
-        simulation="$(arg gazebo_classic)">
-        <origin xyz="0.53 0.33 0.1145" rpy="${PI} 0 ${PI/4}"/>
-    </xacro:sensor_sick_s300>
-    <xacro:sensor_sick_s300
-        frame_prefix="$(arg prefix)rear_laser_"
-        parent="$(arg prefix)chassis_link"
-        node_namespace="$(arg namespace)"
-        node_name="rear_laser"
-        simulation="$(arg gazebo_classic)">
-        <origin xyz="-0.53 -0.33 0.1145" rpy="${PI} 0 ${-PI*3/4}"/>
-    </xacro:sensor_sick_s300>
-	<!-- Controllers -->
-	<xacro:if value="$(arg gazebo_classic)">
-		<xacro:rbvogui_gz_classic_control namespace="$(arg namespace)" prefix="$(arg prefix)"/>
-        <xacro:ros_planar_move_gazebo_classic/>
-	</xacro:if>
+        gazebo_classic="$(arg gazebo_classic)"
+        gazebo_ignition="$(arg gazebo_ignition)">
+        <origin
+            xyz="${rear_rgbd_camera_offset_x} ${rear_rgbd_camera_offset_y} ${rear_rgbd_camera_offset_z}"
+            rpy="0 0 -${PI}" />
+    </xacro:sensor_intel_realsense_d435>
+    <!-- Controllers -->
+    <xacro:if value="$(arg gazebo_classic)">
+        <xacro:rbvogui_gz_classic_control namespace="$(arg namespace)" prefix="$(arg prefix)" />
+        <xacro:ros_planar_move_gazebo_classic />
+    </xacro:if>
+    <xacro:if value="$(arg gazebo_ignition)">
+        <xacro:rbvogui_gz_ignition_control namespace="$(arg namespace)" prefix="$(arg prefix)" />
+    </xacro:if>
     <xacro:unless value="$(arg gazebo_classic)">
-        <xacro:rbvogui_base_hw_controller/>
+        <xacro:unless value="$(arg gazebo_ignition)">
+            <xacro:rbvogui_base_hw_controller />
+        </xacro:unless>
     </xacro:unless>
 </robot>

File: Robotnik_ws/src/robot_description/urdf/bases/rbvogui/rbvogui_base.urdf.xacro (robot description, xacro)
@@ -23,14 +23,14 @@
         <!-- Here we create the robot elements using the xacro:macros imported at the beggining of this file -->
         <xacro:rbvogui_body prefix="${prefix}" hq="${hq}"/>
-        <xacro:steering_wheel robot_id="${prefix}front_right" parent="${prefix}base_link" reflect="false" hq="${hq}">
+        <xacro:steering_wheel prefix="${prefix}front_right_" parent="${prefix}base_link" reflect="false" hq="${hq}">
             <origin xyz="${wheel_offset_x} -${wheel_offset_y} ${wheel_offset_z}" rpy="0 0 0"/>
         </xacro:steering_wheel>
-        <xacro:steering_wheel robot_id="${prefix}front_left" parent="${prefix}base_link" reflect="true" hq="${hq}">
+        <xacro:steering_wheel prefix="${prefix}front_left_" parent="${prefix}base_link" reflect="true" hq="${hq}">
             <origin xyz="${wheel_offset_x} ${wheel_offset_y} ${wheel_offset_z}" rpy="0 0 0"/>
         </xacro:steering_wheel>
-        <xacro:steering_wheel robot_id="${prefix}back_left" parent="${prefix}base_link" reflect="true" hq="${hq}">
+        <xacro:steering_wheel prefix="${prefix}back_left_" parent="${prefix}base_link" reflect="true" hq="${hq}">
             <origin xyz="-${wheel_offset_x} ${wheel_offset_y} ${wheel_offset_z}" rpy="0 0 0"/>
         </xacro:steering_wheel>
-        <xacro:steering_wheel robot_id="${prefix}back_right" parent="${prefix}base_link" reflect="false" hq="${hq}">
+        <xacro:steering_wheel prefix="${prefix}back_right_" parent="${prefix}base_link" reflect="false" hq="${hq}">
             <origin xyz="-${wheel_offset_x} -${wheel_offset_y} ${wheel_offset_z}" rpy="0 0 0"/>
         </xacro:steering_wheel>

File: Robotnik_ws/src/robot_description/urdf/wheels/steering_wheel/steering_wheel.urdf.xacro (robot description, xacro)
@@ -6,5 +6,5 @@
   <xacro:property name="wheel_width" value="0.1375" />
   <xacro:property name="wheel_mass" value="5.0" />
-  <xacro:macro name="steering_wheel" params="robot_id parent *origin reflect hq">
+  <xacro:macro name="steering_wheel" params="prefix parent *origin reflect hq">
     <xacro:macro name="cylinder_inertia" params="m r h">
       <inertia ixx="${m*(3*r*r+h*h)/12}" ixy = "0" ixz = "0" iyy="${m*(3*r*r+h*h)/12}" iyz = "0" izz="${m*r*r/2}" />
@@ -16,13 +16,13 @@
     <xacro:property name="steer_joint_effort_limit" value="200.0" />
     <xacro:property name="steer_joint_velocity_limit" value="100.0" />
-    <joint name="${robot_id}_steering_joint" type="revolute">
+    <joint name="${prefix}steering_joint" type="revolute">
       <parent link="${parent}"/>
-      <child link="${robot_id}_base_wheel"/>
+      <child link="${prefix}base_wheel"/>
       <xacro:insert_block name="origin" />
-      <axis xyz="0 0 1" rpy="0 0 0" />
+      <axis xyz="0 0 1"/>
       <limit effort="${steer_joint_effort_limit}" velocity="${steer_joint_velocity_limit}" lower="-3.00" upper="3.00"/>
       <dynamics damping="${steer_joint_damping}" friction="${steer_joint_friction}"/>
     </joint>
-    <link name="${robot_id}_base_wheel">
+    <link name="${prefix}base_wheel">
       <visual>
         <xacro:if value="${hq}">
@@ -74,6 +74,6 @@
       </inertial>
     </link>
-    <xacro:gazebo_steering_frame_physics name="${robot_id}_base_wheel"/>
-    <xacro:rubber_wheel robot_id="${robot_id}" parent="${robot_id}_base_wheel" reflect="${reflect}" hq="${hq}" rubber_wheel_radius="${wheel_radius}" rubber_wheel_width="${wheel_width}" rubber_wheel_mass="${wheel_mass}">
+    <xacro:gazebo_steering_frame_physics name="${prefix}base_wheel"/>
+    <xacro:rubber_wheel prefix="${prefix}" parent="${prefix}base_wheel" reflect="${reflect}" hq="${hq}" rubber_wheel_radius="${wheel_radius}" rubber_wheel_width="${wheel_width}" rubber_wheel_mass="${wheel_mass}">
         <origin xyz="0 0 0" rpy="0 0 0"/>
     </xacro:rubber_wheel>

File: Robotnik_ws/src/robotnik_sensors/robotnik_sensors/urdf/2d_lidar/sick_s300.urdf.xacro (robot description, xacro)
@@ -1,9 +1,11 @@
 <?xml version="1.0"?>
 <robot name="sensor_sick_s300" xmlns:xacro="http://wiki.ros.org/xacro">
+  <xacro:include filename="$(find robotnik_sensors)/urdf/2d_lidar/lidar_2d_plugin.urdf.xacro" />
   <xacro:macro name="sensor_sick_s300"
                params="frame_prefix
                        parent
                        *origin
-                       simulation:=false
+                       gazebo_classic:=false
+                       gazebo_ignition:=false
                        node_name:=sick_s300
                        node_namespace:=${None}
@@ -44,50 +46,19 @@
     </joint>
     <link name="${frame_prefix}link"/>
-    <xacro:if value="${simulation}">
-      <xacro:sensor_sick_s300_gazebo/>
-    </xacro:if>
-  </xacro:macro>
-  <xacro:macro name="sensor_sick_s300_gazebo">
-      <xacro:if value="${gpu}">
-        <xacro:property name="ray_type" value="gpu_ray" />
-      </xacro:if>
-      <xacro:unless value="${gpu}">
-        <xacro:property name="ray_type" value="ray" />
-      </xacro:unless>
-      <gazebo reference="${frame_prefix}link">
-        <sensor type="${ray_type}" name="${frame_prefix}sensor">
-          <pose>0.0 0.0 0.0 0.0 0.0 0.0</pose>
-          <visualize>false</visualize>
-          <update_rate>25.0</update_rate>
-          <ray>
-            <scan>
-              <horizontal>
-                <samples>270</samples>
-                <resolution>1</resolution>
-                <min_angle>${-radians(135)}</min_angle>
-                <max_angle>${radians(135)}</max_angle>
-              </horizontal>
-            </scan>
-            <range>
-              <min>0.05</min>
-              <max>10.0</max>
-              <resolution>0.00575</resolution>
-            </range>
-            <noise>
-              <type>gaussian</type>
-              <mean>0.0</mean>
-              <stddev>0.01</stddev>
-            </noise>
-          </ray>
-          <plugin name="${node_name}" filename="libgazebo_ros_ray_sensor.so">
-            <ros>
-              <namespace>${node_namespace}</namespace>
-              <remapping>~/out:=~/scan</remapping>
-            </ros>
-            <output_type>sensor_msgs/LaserScan</output_type>
-            <frame_name>${frame_prefix}link</frame_name>
-          </plugin>
-        </sensor>
-      </gazebo>
+    <xacro:lidar_2d_plugin
+      node_namespace="${node_namespace}"
+      node_name="${node_name}"
+      gazebo_classic="${gazebo_classic}"
+      gazebo_ignition="${gazebo_ignition}"
+      min_range="0.05"
+      max_range="10.0"
+      min_angle="${-radians(130)}"
+      max_angle="${radians(130)}"
+      frame_link="${frame_prefix}link"
+      rate="25.0"
+      resolution="0.00575"
+      samples="270"
+    >
+    </xacro:lidar_2d_plugin>
   </xacro:macro>
 </robot>

File: Robotnik_ws/src/robotnik_sensors/robotnik_sensors/urdf/3d_lidar/robosense_helios_16p.urdf.xacro (robot description, xacro)
@@ -57,6 +57,6 @@
       max_angle="85"
       frame_link="${frame_prefix}link"
-      rate="10"
-      horizontal_samples="1200"
+      rate="5"
+      horizontal_samples="600"
       vertical_samples="16"
     >

File: Robotnik_ws/src/robotnik_sensors/robotnik_sensors/urdf/camera/camera_plugin.urdf.xacro (robot description, xacro)
@@ -66,9 +66,4 @@
               <far>${max_depth}</far>
             </clip>
-            <noise>
-                <type>gaussian</type>
-                <mean>0.0</mean>
-                <stddev>0.05</stddev>
-            </noise>
             </camera>
             <always_on>1</always_on>

File: Robotnik_ws/src/robotnik_sensors/robotnik_sensors/urdf/depth/depth_camera_plugin.urdf.xacro (robot description, xacro)
@@ -74,12 +74,7 @@
               <far>${max_depth}</far>
             </clip>
-            <noise>
-              <type>gaussian</type>
-              <mean>0.0</mean>
-              <stddev>0.100</stddev>
-            </noise>
           </camera>
           <always_on>1</always_on>
-          <update_rate>90</update_rate>
+          <update_rate>${rate}</update_rate>
           <visualize>false</visualize>
           <topic>${node_namespace}/${node_name}/depth/image_raw</topic>

File: Robotnik_ws/src/robotnik_sensors/robotnik_sensors/urdf/depth/intel_realsense_d435.urdf.xacro (robot description, xacro)
@@ -145,11 +145,11 @@
         optical_frame="${frame_prefix}infra1_optical_frame"
         reference_frame="${frame_prefix}infra2_frame"
-        horizontal_fov="85.2"
-        vertical_fov="48"
-        video_width="1280"
-        video_height="720"
+        horizontal_fov="60"
+        vertical_fov="30"
+        video_width="640"
+        video_height="480"
         min_depth="0.1"
         max_depth="100"
-        rate="30"
+        rate="5"
       >
       </xacro:irred_camera_plugin>
@@ -162,11 +162,11 @@
         optical_frame="${frame_prefix}infra2_optical_frame"
         reference_frame="${frame_prefix}infra2_frame"
-        horizontal_fov="85.2"
-        vertical_fov="48"
-        video_width="1280"
-        video_height="720"
+        horizontal_fov="60"
+        vertical_fov="30"
+        video_width="640"
+        video_height="480"
         min_depth="0.1"
         max_depth="100"
-        rate="30"
+        rate="5"
       >
       </xacro:irred_camera_plugin>
@@ -179,11 +179,11 @@
         optical_frame="${frame_prefix}depth_optical_frame"
         reference_frame="${frame_prefix}depth_frame"
-        horizontal_fov="85.2"
-        vertical_fov="48"
-        video_width="1280"
-        video_height="720"
+        horizontal_fov="60"
+        vertical_fov="30"
+        video_width="640"
+        video_height="480"
         min_depth="0.1"
         max_depth="100"
-        rate="30"
+        rate="5"
       >
       </xacro:depth_camera_plugin>

File: Robotnik_ws/src/robotnik_sensors/robotnik_sensors/urdf/depth/irred_camera_plugin.urdf.xacro (robot description, xacro)
@@ -66,9 +66,4 @@
               <far>${max_depth}</far>
             </clip>
-            <noise>
-                <type>gaussian</type>
-                <mean>0.0</mean>
-                <stddev>0.05</stddev>
-            </noise>
             </camera>
             <always_on>1</always_on>
