Commit message: Prefix Tfs en Ignition

File: Robotnik_ws/src/robot_description/simulators/gazebo_ignition/rbrobout/rbrobout_control.urdf.xacro (robot description, xacro)
@@ -27,9 +27,9 @@
               <plugin>ign_ros2_control/IgnitionSystem</plugin>
           </hardware>
-          <xacro:ros2_joint interface="velocity" jmin="-10" jmax="10" name="${prefix}front_left_wheel_joint"/>
-          <xacro:ros2_joint interface="velocity" jmin="-10" jmax="10" name="${prefix}front_right_wheel_joint"/>
-          <xacro:ros2_joint interface="velocity" jmin="-20" jmax="20" name="${prefix}back_left_wheel_joint"/>
-          <xacro:ros2_joint interface="velocity" jmin="-20" jmax="20" name="${prefix}back_right_wheel_joint"/>
-          <xacro:ros2_joint interface="position" jmin="-20" jmax="20" name="${prefix}lift_ewellix_lift_top_joint"/>
+          <xacro:ros2_joint interface="velocity" jmin="-10" jmax="10" name="robot_front_left_wheel_joint"/>
+          <xacro:ros2_joint interface="velocity" jmin="-10" jmax="10" name="robot_front_right_wheel_joint"/>
+          <xacro:ros2_joint interface="velocity" jmin="-20" jmax="20" name="robot_back_left_wheel_joint"/>
+          <xacro:ros2_joint interface="velocity" jmin="-20" jmax="20" name="robot_back_right_wheel_joint"/>
+          <xacro:ros2_joint interface="position" jmin="-20" jmax="20" name="robot_lift_ewellix_lift_top_joint"/>
         </ros2_control>
     </xacro:macro>

File: Robotnik_ws/src/robot_description/simulators/gazebo_ignition/rbwatcher/rbwatcher_control.urdf.xacro (robot description, xacro)
@@ -27,10 +27,10 @@
               <plugin>ign_ros2_control/IgnitionSystem</plugin>
           </hardware>
-          <xacro:ros2_joint interface="velocity" jmin="-10" jmax="10" name="${prefix}front_left_wheel_joint"/>
-          <xacro:ros2_joint interface="velocity" jmin="-10" jmax="10" name="${prefix}front_right_wheel_joint"/>
-          <xacro:ros2_joint interface="velocity" jmin="-20" jmax="20" name="${prefix}back_left_wheel_joint"/>
-          <xacro:ros2_joint interface="velocity" jmin="-20" jmax="20" name="${prefix}back_right_wheel_joint"/>
-          <xacro:ros2_joint interface="position" jmin="-20" jmax="20" name="${prefix}top_ptz_camera_pan_joint"/>
-          <xacro:ros2_joint interface="position" jmin="-20" jmax="20" name="${prefix}top_ptz_camera_tilt_joint"/>
+          <xacro:ros2_joint interface="velocity" jmin="-10" jmax="10" name="robot_front_left_wheel_joint"/>
+          <xacro:ros2_joint interface="velocity" jmin="-10" jmax="10" name="robot_front_right_wheel_joint"/>
+          <xacro:ros2_joint interface="velocity" jmin="-20" jmax="20" name="robot_back_left_wheel_joint"/>
+          <xacro:ros2_joint interface="velocity" jmin="-20" jmax="20" name="robot_back_right_wheel_joint"/>
+          <xacro:ros2_joint interface="position" jmin="-20" jmax="20" name="robot_top_ptz_camera_pan_joint"/>
+          <xacro:ros2_joint interface="position" jmin="-20" jmax="20" name="robot_top_ptz_camera_tilt_joint"/>
         </ros2_control>
     </xacro:macro>

File: Robotnik_ws/src/robot_description/urdf/bases/rbrobout/rbrobout_base.urdf.xacro (robot description, xacro)
@@ -25,14 +25,14 @@
 		<xacro:rbrobout_body prefix="${prefix}" />
 		<!-- Wheels -->
-		<xacro:rbrobout_omni_wheel prefix="${prefix}front_right" parent="${prefix}base_link" reflect="false" hq="${hq}">
+		<xacro:rbrobout_omni_wheel prefix1="${prefix}" prefix2="front_right" parent="${prefix}base_link" reflect="false" hq="${hq}">
 			<origin xyz="${wheel_offset_x} -${wheel_offset_y} ${wheel_offset_z}" rpy="0 0 0"/>
 		</xacro:rbrobout_omni_wheel>
-		<xacro:rbrobout_omni_wheel prefix="${prefix}front_left" parent="${prefix}base_link" reflect="true" hq="${hq}">
+		<xacro:rbrobout_omni_wheel prefix1="${prefix}" prefix2="front_left" parent="${prefix}base_link" reflect="true" hq="${hq}">
 			<origin xyz="${wheel_offset_x} ${wheel_offset_y} ${wheel_offset_z}" rpy="0 0 0"/>
 		</xacro:rbrobout_omni_wheel>
-		<xacro:rbrobout_omni_wheel prefix="${prefix}back_left" parent="${prefix}base_link" reflect="true" hq="${hq}">
+		<xacro:rbrobout_omni_wheel prefix1="${prefix}" prefix2="back_left" parent="${prefix}base_link" reflect="true" hq="${hq}">
 			<origin xyz="-${wheel_offset_x} ${wheel_offset_y} ${wheel_offset_z}" rpy="0 0 0"/>
 		</xacro:rbrobout_omni_wheel>
-		<xacro:rbrobout_omni_wheel prefix="${prefix}back_right" parent="${prefix}base_link" reflect="false" hq="${hq}">
+		<xacro:rbrobout_omni_wheel prefix1="${prefix}" prefix2="back_right" parent="${prefix}base_link" reflect="false" hq="${hq}">
 			<origin xyz="-${wheel_offset_x} -${wheel_offset_y} ${wheel_offset_z}" rpy="0 0 0"/>
 		</xacro:rbrobout_omni_wheel>

File: Robotnik_ws/src/robot_description/urdf/bases/rbwatcher/rbwatcher_base.urdf.xacro (robot description, xacro)
@@ -8,5 +8,5 @@
 	<xacro:include filename="$(find robot_description)/urdf/bodies/rbwatcher/rbwatcher_body.urdf.xacro" />
 	<!-- Import RB-Watcher wheels -->
-  	<xacro:include filename="$(find robot_description)/urdf/wheels/rubber_wheel/rubber_wheel.urdf.xacro" />
+  	<xacro:include filename="$(find robot_description)/urdf/wheels/rubber_wheel/rbwatcher_rubber_wheel.urdf.xacro" />
   	<xacro:include filename="$(find robot_description)/urdf/wheels/omni_wheel/omni_wheel.urdf.xacro" />
 	<!-- Import all available sensors -->
@@ -35,5 +35,6 @@
 		<!-- Wheels -->
 		<xacro:rubber_wheel
-	            prefix="${prefix}front_right"
+	            prefix1="${prefix}"
+	            prefix2="front_right"
 	            parent="${prefix}base_link"
 	            reflect="false" hq="${hq}"
@@ -45,5 +46,6 @@
 		</xacro:rubber_wheel>
 		<xacro:rubber_wheel
-	            prefix="${prefix}front_left"
+	            prefix1="${prefix}"
+	            prefix2="front_left"
 	            parent="${prefix}base_link"
 	            reflect="false" hq="${hq}"
@@ -55,5 +57,6 @@
 		</xacro:rubber_wheel>
 		<xacro:rubber_wheel
-	            prefix="${prefix}back_right"
+	            prefix1="${prefix}"
+	            prefix2="back_right"
 	            parent="${prefix}base_link"
 	            reflect="false" hq="${hq}"
@@ -65,5 +68,6 @@
 		</xacro:rubber_wheel>
 		<xacro:rubber_wheel
-	            prefix="${prefix}back_left"
+	            prefix1="${prefix}"
+	            prefix2="back_left"
 	            parent="${prefix}base_link"
 	            reflect="false" hq="${hq}"

File: Robotnik_ws/src/robot_description/urdf/wheels/omni_wheel/rbrobout_omni_wheel.urdf.xacro (robot description, xacro)
@@ -11,8 +11,8 @@
               izz="${m*(3*r*r+h*h)/12}" />
   </xacro:macro>
-  <xacro:macro name="rbrobout_omni_wheel" params="prefix parent *origin reflect hq">
-    <joint name="${prefix}_wheel_joint" type="continuous">
+  <xacro:macro name="rbrobout_omni_wheel" params="prefix1 prefix2 parent *origin reflect hq">
+    <joint name="robot_${prefix2}_wheel_joint" type="continuous">
       <parent link="${parent}"/>
-      <child link="${prefix}_wheel_link"/>
+      <child link="${prefix1}${prefix2}_wheel_link"/>
       <xacro:insert_block name="origin" />
       <axis xyz="0 1 0" rpy="0 0 0" />
@@ -20,5 +20,5 @@
       <joint_properties damping="0.0" friction="0.0"/>
     </joint>
-    <link name="${prefix}_wheel_link">
+    <link name="${prefix1}${prefix2}_wheel_link">
       <visual>
         <xacro:if value="${hq}">
@@ -50,5 +50,5 @@
       </inertial>
     </link>
-    <gazebo reference="${prefix}wheel_link">
+    <gazebo reference="${prefix1}${prefix2}_wheel_link">
       <mu1>0.0</mu1>
       <mu2>0.0</mu2>

File: Robotnik_ws/src/robotnik_sensors/robotnik_sensors/urdf/link_750_nh.urdf.xacro (robot description, xacro)
@@ -38,5 +38,5 @@
       </collision>
     </link>
-    <joint name="${prefix}_pan_joint" type="revolute">
+    <joint name="robot_top_ptz_camera_pan_joint" type="revolute">
       <axis xyz="0 0 1"/>
       <origin xyz="0.0 0.0 0.0318" rpy="0 0 0"/>
@@ -73,5 +73,5 @@
     <transmission name="${prefix}_pan_trans">
       <type>transmission_interface/SimpleTransmission</type>
-      <joint name="${prefix}_pan_joint">
+      <joint name="robot_top_ptz_camera_pan_joint">
         <hardwareInterface>hardware_interface/PositionJointInterface</hardwareInterface>
       </joint>
@@ -81,5 +81,5 @@
       </actuator>
     </transmission>
-    <joint name="${prefix}_tilt_joint" type="revolute">
+    <joint name="robot_top_ptz_camera_tilt_joint" type="revolute">
       <axis xyz="0 0 1"/>
       <origin xyz="0.0 0.0 0.102" rpy="${PI/2} 0 0"/>
@@ -115,5 +115,5 @@
     <transmission name="${prefix}_tilt_trans">
       <type>transmission_interface/SimpleTransmission</type>
-      <joint name="${prefix}_tilt_joint">
+      <joint name="robot_top_ptz_camera_tilt_joint">
         <hardwareInterface>hardware_interface/PositionJointInterface</hardwareInterface>
       </joint>
