Commit message: Odometria arreglada
La odometria se ha corregido y ahora cuadra completamente con el robot, por otro lado, el robot se puede de forma correcta hacia delante y hacia atrás, pero no gira aún.

File: Robotnik_ws/src/robot_description/robots/rbrobout/rbrobout.urdf.xacro (robot description, xacro)
@@ -92,5 +92,6 @@
     <xacro:if value="${simulator == 'gazebo_ignition'}">
         <xacro:rbrobout_gz_ignition_control namespace="$(arg namespace)" prefix="$(arg prefix)"/>
-        <xacro:ros_diff_move_gazebo_ignition prefix="$(arg prefix)"/>
+        <xacro:ros_diff_move_gazebo_ignition_front prefix="$(arg prefix)"/>
+        <xacro:ros_diff_move_gazebo_ignition_rear prefix="$(arg prefix)"/>
     </xacro:if>
     <xacro:if value="${simulator == 'none'}">

File: Robotnik_ws/src/robot_description/simulators/gazebo_ignition/rbrobout/rbrobout_control.urdf.xacro (robot description, xacro)
@@ -34,5 +34,5 @@
         </ros2_control>
     </xacro:macro>
-    <xacro:macro name="ros_diff_move_gazebo_ignition" params="prefix">
+    <xacro:macro name="ros_diff_move_gazebo_ignition_front" params="prefix">
         <gazebo>
           <plugin
@@ -40,7 +40,7 @@
              name="ignition::gazebo::systems::DiffDrive">
              <left_joint>${prefix}front_left_wheel_joint</left_joint>
-             <right_joint>${prefix}front_right_wheel_joint</right_joint>
-             <wheel_separation>1.2</wheel_separation>
-             <wheel_radius>0.573</wheel_radius>
+	     <right_joint>${prefix}front_right_wheel_joint</right_joint>
+             <wheel_separation>0.573</wheel_separation>
+             <wheel_radius>0.127</wheel_radius>
              <odom_publish_frequency>1</odom_publish_frequency>
              <topic>cmd_vel</topic>
@@ -50,3 +50,21 @@
         </gazebo>
     </xacro:macro>
+    <xacro:macro name="ros_diff_move_gazebo_ignition_rear" params="prefix">
+        <gazebo>
+          <plugin
+             filename="libignition-gazebo-diff-drive-system.so"
+             name="ignition::gazebo::systems::DiffDrive">
+	     <left_joint>${prefix}back_left_wheel_joint</left_joint>
+	     <right_joint>${prefix}back_right_wheel_joint</right_joint>
+             <wheel_separation>0.573</wheel_separation>
+             <wheel_radius>0.127</wheel_radius>
+             <odom_publish_frequency>0</odom_publish_frequency>
+             <publish_odom>false</publish_odom>
+             <publish_odom_tf>false</publish_odom_tf>
+             <topic>cmd_vel_rear</topic>
+             <frame_id>robot_odom</frame_id>
+             <child_frame_id>robot_base_footprint</child_frame_id>
+          </plugin>
+        </gazebo>
+    </xacro:macro>
 </robot>

File: Robotnik_ws/src/robot_description/urdf/wheels/omni_wheel/rbrobout_omni_wheel.urdf.xacro (robot description, xacro)
@@ -51,8 +51,8 @@
     </link>
     <gazebo reference="${prefix}_wheel_link">
-      <mu1>0.0</mu1>
-      <mu2>0.0</mu2>
-      <kp>0</kp>
-      <kd>0</kd>
+      <mu1>0.90</mu1>
+      <mu2>0.85</mu2>
+      <kp>2.75e6</kp>
+      <kd>8.25e1</kd>
       <fdir1>0 0 0</fdir1>
     </gazebo>

Commit message: Arreglo de los tfs móviles del Rbwatcher y acercamiento de la estructura del launcher a la de robotnik

File: Robotnik_ws/src/robot_description/robots/rbrobout/rbrobout.urdf.xacro (robot description, xacro)
@@ -36,6 +36,6 @@
         parent="$(arg prefix)base_link"
         node_namespace="$(arg namespace)"
-        simulation="$(arg gazebo_classic)"
-        simulator="$(arg simulator)">
+        gazebo_classic="$(arg gazebo_classic)"
+        gazebo_ignition="$(arg gazebo_ignition)">
         <origin xyz="${imu_offset_x} ${imu_offset_y} ${imu_offset_z}" rpy="0 0 0"/>
     </xacro:sensor_vectornav>
@@ -46,6 +46,6 @@
         node_namespace="$(arg namespace)"
         node_name="front_camera"
-        simulator="$(arg simulator)"
-        simulation="$(arg gazebo_classic)"
+        gazebo_ignition="$(arg gazebo_ignition)"
+        gazebo_classic="$(arg gazebo_classic)"
         topic_prefix="front_rgbd_camera">
         <origin xyz="${front_rgbd_camera_offset_x} ${front_rgbd_camera_offset_y} ${front_rgbd_camera_offset_z}" rpy="0 0 0"/>
@@ -57,6 +57,6 @@
         node_namespace="$(arg namespace)"
         node_name="rear_camera"
-        simulator="$(arg simulator)"
-        simulation="$(arg gazebo_classic)"
+        gazebo_ignition="$(arg gazebo_ignition)"
+        gazebo_classic="$(arg gazebo_classic)"
         topic_prefix="rear_rgbd_camera">
         <origin xyz="${rear_rgbd_camera_offset_x} ${rear_rgbd_camera_offset_y} ${rear_rgbd_camera_offset_z}" rpy="0 ${PI} 0"/>
@@ -68,7 +68,6 @@
         node_namespace="$(arg namespace)"
         node_name="front_laser"
-        simulation="$(arg gazebo_classic)"
-        simulator="$(arg simulator)"
-        topic_prefix="front_laser">
+        gazebo_classic="$(arg gazebo_classic)"
+        gazebo_ignition="$(arg gazebo_ignition)">
         <origin xyz="${front_laser_offset_x} ${front_laser_offset_y} ${front_laser_offset_z}" rpy="0 0 ${1/4*PI}"/>
     </xacro:sensor_sick_microscan3>
@@ -79,22 +78,22 @@
         node_namespace="$(arg namespace)"
         node_name="rear_laser"
-        simulation="$(arg gazebo_classic)"
-        simulator="$(arg simulator)"
-        topic_prefix="rear_laser">
+        gazebo_classic="$(arg gazebo_classic)"
+        gazebo_ignition="$(arg gazebo_ignition)">
         <origin xyz="${rear_laser_offset_x} ${rear_laser_offset_y} ${rear_laser_offset_z}" rpy="0 0 ${-3/4*PI}"/>
     </xacro:sensor_sick_microscan3>
     <!-- Controllers -->
-    <xacro:property name="simulator" value="$(arg simulator)"/>
-    <xacro:if value="${simulator == 'gazebo_classic'}">
+    <xacro:if value="$(arg gazebo_classic)">
         <xacro:rbrobout_gz_classic_control namespace="$(arg namespace)" prefix="$(arg prefix)"/>
         <xacro:ros_planar_move_gazebo_classic/>
     </xacro:if>
-    <xacro:if value="${simulator == 'gazebo_ignition'}">
+    <xacro:if value="$(arg gazebo_ignition)">
         <xacro:rbrobout_gz_ignition_control namespace="$(arg namespace)" prefix="$(arg prefix)"/>
         <xacro:ros_diff_move_gazebo_ignition_front prefix="$(arg prefix)"/>
         <xacro:ros_diff_move_gazebo_ignition_rear prefix="$(arg prefix)"/>
     </xacro:if>
-    <xacro:if value="${simulator == 'none'}">
-        <xacro:rbrobout_base_hw_controller/>
-    </xacro:if>
+    <xacro:unless value="$(arg gazebo_classic)">
+        <xacro:unless value="$(arg gazebo_ignition)">
+            <xacro:rbrobout_base_hw_controller/>
+        </xacro:unless>
+    </xacro:unless>
 </robot>

File: Robotnik_ws/src/robot_description/robots/rbwatcher/rbwatcher.urdf.xacro (robot description, xacro)
@@ -21,5 +21,5 @@
 	<xacro:arg name="namespace" default="robot"/>
         <xacro:arg name="gazebo_classic" default="false"/>
-        <xacro:arg name="simulator" default="gazebo_ignition"/>
+        <xacro:arg name="gazebo_ignition" default="false"/>
     <xacro:macro name="rbwatcher" params="prefix publish_bf hq kinematics:=skid leika:=false">
 		<xacro:property name="top_structure_mesh" value="robot_description/meshes/structures/rbwatcher/rbwatcher_top_structure" />
@@ -43,6 +43,6 @@
         parent="$(arg prefix)base_link"
         node_namespace="$(arg namespace)"
-        simulation="$(arg gazebo_classic)"
-        simulator="$(arg simulator)">
+        gazebo_classic="$(arg gazebo_classic)"
+        gazebo_ignition="$(arg gazebo_ignition)">
     	  	<origin xyz="-0.03534 0.132 0.16109" rpy="0 0 0"/>
     	</xacro:sensor_vectornav>
@@ -53,6 +53,6 @@
         node_namespace="$(arg namespace)"
         node_name="front_camera"
-        simulator="$(arg simulator)"
-        simulation="$(arg gazebo_classic)"
+        gazebo_classic="$(arg gazebo_classic)"
+        gazebo_ignition="$(arg gazebo_ignition)"
         topic_prefix="front_rgbd_camera">
 	<origin xyz="0.29881 0.0 0.15243" rpy="0 0 0"/>
@@ -63,6 +63,6 @@
         node_namespace="$(arg namespace)"
         node_name="rear_camera"
-        simulator="$(arg simulator)"
-        simulation="$(arg gazebo_classic)"
+        gazebo_classic="$(arg gazebo_classic)"
+        gazebo_ignition="$(arg gazebo_ignition)"
         topic_prefix="rear_rgbd_camera">
 		<origin xyz="-0.308 0.0 0.18308" rpy="0 ${-PI} 0"/>
@@ -73,5 +73,5 @@
         </xacro:sensor_ublox>
     	<!-- LIDAR -->
-    	<xacro:sensor_robosense_helios_16p frame_prefix="$(arg prefix)top_3d_laser" node_namespace="$(arg namespace)" topic_prefix="top_3d_laser" parent="$(arg prefix)base_link" gpu="$(arg gpu)" simulation="$(arg gazebo_classic)">
+    	<xacro:sensor_robosense_helios_16p frame_prefix="$(arg prefix)top_3d_laser" node_namespace="$(arg namespace)" topic_prefix="top_3d_laser" parent="$(arg prefix)base_link" gpu="$(arg gpu)" simulation="$(arg gazebo_ignition)">
     	  	<origin xyz="-0.11924 0.0 0.38609" rpy="0 0 0"/>
     	</xacro:sensor_robosense_helios_16p>

File: Robotnik_ws/src/robot_description/simulators/gazebo_ignition/rbwatcher/rbwatcher_control.urdf.xacro (robot description, xacro)
@@ -31,5 +31,6 @@
           <xacro:ros2_joint interface="velocity" jmin="-20" jmax="20" name="${prefix}back_left_wheel_joint"/>
           <xacro:ros2_joint interface="velocity" jmin="-20" jmax="20" name="${prefix}back_right_wheel_joint"/>
-          <xacro:ros2_joint interface="position" jmin="-20" jmax="20" name="${prefix}lift_ewellix_lift_top_joint"/>
+          <xacro:ros2_joint interface="position" jmin="-20" jmax="20" name="${prefix}top_ptz_camera_pan_joint"/>
+          <xacro:ros2_joint interface="position" jmin="-20" jmax="20" name="${prefix}top_ptz_camera_tilt_joint"/>
         </ros2_control>
     </xacro:macro>

File: Robotnik_ws/src/robotnik_sensors/robotnik_sensors/urdf/2d_lidar/sick_microscan3.urdf.xacro (robot description, xacro)
@@ -1,13 +1,14 @@
 <?xml version="1.0"?>
 <robot name="sensor_sick_microscan3" xmlns:xacro="http://wiki.ros.org/xacro">
+  <xacro:include filename="$(find robotnik_sensors)/urdf/2d_lidar/lidar_2d_plugin.urdf.xacro" />
   <xacro:macro name="sensor_sick_microscan3"
                params="frame_prefix
                        parent
                        *origin
-                       simulation:=false
-                       simulator:=gazebo_classic
+                       gazebo_classic:=false
+                       gazebo_ignition:=false
                        node_name:=sick_microscan3
                        node_namespace:=${None}
-                       topic_prefix:=/scan
+                       topic_prefix:=~/
                        gpu:=false">
     <!-- node_namespace is used from node_name if not set -->
@@ -46,93 +47,19 @@
     <link name="${frame_prefix}link"/>
     <!-- sick_microscan3 sensor for simulation -->
-    <xacro:if value="${simulator == 'gazebo_classic'}">
-      <xacro:sensor_sick_microscan3_gazebo />
-    </xacro:if>
-    <xacro:if value="${simulator == 'gazebo_ignition'}">
-      <xacro:sensor_sick_microscan3_ignition />
-    </xacro:if>
-  </xacro:macro>
-  <xacro:macro name="sensor_sick_microscan3_gazebo">
-    <xacro:if value="${gpu}">
-        <xacro:property name="ray_type" value="gpu_ray" />
-      </xacro:if>
-      <xacro:unless value="${gpu}">
-        <xacro:property name="ray_type" value="ray" />
-      </xacro:unless>
-      <gazebo reference="${frame_prefix}link">
-        <sensor type="${ray_type}" name="${frame_prefix}sensor">
-          <pose>0.0 0.0 0.0 0.0 0.0 0.0</pose>
-          <visualize>false</visualize>
-          <update_rate>20.0</update_rate>
-          <ray>
-            <scan>
-              <horizontal>
-                <samples>700</samples>
-                <resolution>1</resolution>
-                <min_angle>-2.35</min_angle>
-                <max_angle>2.35</max_angle>
-              </horizontal>
-            </scan>
-            <range>
-              <min>0.05</min>
-              <max>64.0</max>
-              <resolution>0.00575</resolution>
-            </range>
-            <noise>
-              <type>gaussian</type>
-              <mean>0.0</mean>
-              <stddev>0.01</stddev>
-            </noise>
-          </ray>
-          <always_on>true</always_on>
-          <plugin name="${node_name}" filename="libgazebo_ros_ray_sensor.so">
-            <ros>
-              <namespace>${node_namespace}</namespace>
-              <remapping>~/out:=~/scan</remapping>
-            </ros>
-            <output_type>sensor_msgs/LaserScan</output_type>
-            <frame_name>${frame_prefix}link</frame_name>
-          </plugin>
-        </sensor>
-      </gazebo>
-  </xacro:macro>
-  <xacro:macro name="sensor_sick_microscan3_ignition">
-    <xacro:if value="${gpu}">
-        <xacro:property name="lidar_type" value="gpu_lidar" />
-      </xacro:if>
-      <xacro:unless value="${gpu}">
-        <xacro:property name="lidar_type" value="lidar" />
-      </xacro:unless>
-      <gazebo reference="${frame_prefix}link">
-        <sensor type="gpu_lidar" name="${frame_prefix}sensor">
-          <pose>0.0 0.0 0.0 0.0 0.0 0.0</pose>
-          <frame_id>${frame_prefix}link</frame_id>
-          <topic>${topic_prefix}/scan</topic>
-          <visualize>false</visualize>
-          <update_rate>20.0</update_rate>
-          <ignition_frame_id>${frame_prefix}link</ignition_frame_id>
-          <ray>
-            <scan>
-              <horizontal>
-                <samples>700</samples>
-                <resolution>1</resolution>
-                <min_angle>-2.35</min_angle>
-                <max_angle>2.35</max_angle>
-              </horizontal>
-            </scan>
-            <range>
-              <min>0.05</min>
-              <max>64.0</max>
-              <resolution>0.00575</resolution>
-            </range>
-            <noise>
-              <type>gaussian</type>
-              <mean>0.0</mean>
-              <stddev>0.01</stddev>
-            </noise>
-          </ray>
-          <always_on>true</always_on>
-        </sensor>
-      </gazebo>
+    <xacro:lidar_2d_plugin
+      node_namespace="${node_namespace}"
+      node_name="${node_name}"
+      gazebo_classic="${gazebo_classic}"
+      gazebo_ignition="${gazebo_ignition}"
+      min_range="0.05"
+      max_range="64.0"
+      min_angle="-2.35"
+      max_angle="2.35"
+      frame_link="${frame_prefix}link"
+      rate="30"
+      resolution="0.00575"
+      samples="700"
+    >
+    </xacro:lidar_2d_plugin>
   </xacro:macro>
 </robot>
