Commit message: Arreglo de los tfs móviles del Rbwatcher y acercamiento de la estructura del launcher a la de robotnik

File: Robotnik_ws/src/robotnik_sensors/robotnik_sensors/urdf/depth/intel_realsense_d435.urdf.xacro (robot description, xacro)
@@ -1,10 +1,13 @@
 <?xml version="1.0"?>
 <robot name="sensor_intel_realsense_d435" xmlns:xacro="http://wiki.ros.org/xacro">
+  <xacro:include filename="$(find robotnik_sensors)/urdf/depth/depth_camera_plugin.urdf.xacro" />
+  <xacro:include filename="$(find robotnik_sensors)/urdf/depth/irred_camera_plugin.urdf.xacro" />
+  <xacro:include filename="$(find robotnik_sensors)/urdf/camera/camera_plugin.urdf.xacro" />
   <xacro:macro name="sensor_intel_realsense_d435"
                params="frame_prefix
                        parent
                        *origin
-                       simulation:=false
-                       simulator:=gazebo_classic
+                       gazebo_classic:=false
+                       gazebo_ignition:=false
                        node_name:=realsense_d435
                        node_namespace:=${None}
@@ -65,5 +68,4 @@
     </link>
     <!-- Use the nominal extrinsics between camera frames if the calibrated extrinsics aren't being published. e.g. running the device in simulation  -->
-    <xacro:if value="${simulation}">
       <!-- camera depth joints and links -->
       <joint name="${frame_prefix}depth_joint" type="fixed">
@@ -118,267 +120,72 @@
       </joint>
       <link name="${frame_prefix}color_optical_frame"/>
-      <!-- intel_realsense_d435 sensor for simulation -->
-      <xacro:if value="${simulator == 'gazebo_classic'}">
-        <xacro:intel_realsense_d435_gazebo />
-      </xacro:if>
-      <xacro:if value="${simulator == 'gazebo_ignition'}">
-        <xacro:intel_realsense_d435_ignition />
-      </xacro:if>
-    </xacro:if>
-   </xacro:macro>
-   <xacro:macro name="intel_realsense_d435_gazebo">
-   <gazebo reference="${frame_prefix}color_frame">
-        <sensor name="${node_namespace}color" type="camera">
-          <camera name="${frame_prefix}camera">
-            <horizontal_fov>${radians(69.4)}</horizontal_fov>
-            <image>
-              <width>1920</width>
-              <height>1080</height>
-              <format>RGB_INT8</format>
-            </image>
-            <clip>
-              <near>0.1</near>
-              <far>100</far>
-            </clip>
-            <noise>
-              <type>gaussian</type>
-              <mean>0.0</mean>
-              <stddev>0.007</stddev>
-            </noise>
-          </camera>
-          <always_on>1</always_on>
-          <update_rate>30</update_rate>
-          <visualize>false</visualize>
-          <plugin name="${node_name}_color" filename="libgazebo_ros_camera.so">
-            <ros>
-              <namespace>${node_namespace}/${node_name}</namespace>
-            </ros>
-            <camera_name>${node_name}_color</camera_name>
-            <frame_name>${frame_prefix}color_optical_frame</frame_name>
-          </plugin>
-        </sensor>
-      </gazebo>
-      <gazebo reference="${frame_prefix}infra1_frame">
-        <sensor name="${node_namespace}ired1" type="camera">
-          <camera name="${frame_prefix}camera">
-            <horizontal_fov>${radians(85.2)}</horizontal_fov>
-            <image>
-              <width>1280</width>
-              <height>720</height>
-              <format>L_INT8</format>
-            </image>
-            <clip>
-              <near>0.1</near>
-              <far>100</far>
-            </clip>
-            <noise>
-              <type>gaussian</type>
-              <mean>0.0</mean>
-              <stddev>0.05</stddev>
-            </noise>
-          </camera>
-          <always_on>1</always_on>
-          <update_rate>90</update_rate>
-          <visualize>false</visualize>
-          <plugin name="${node_name}_ired1" filename="libgazebo_ros_camera.so">
-            <ros>
-              <namespace>${node_namespace}/${node_name}</namespace>
-            </ros>
-            <camera_name>${node_name}_ired1</camera_name>
-            <frame_name>${frame_prefix}infra1_optical_frame</frame_name>
-          </plugin>
-        </sensor>
-      </gazebo>
-      <gazebo reference="${frame_prefix}infra2_frame">
-        <sensor name="${node_namespace}ired2" type="camera">
-          <camera name="${frame_prefix}camera">
-            <horizontal_fov>${radians(85.2)}</horizontal_fov>
-            <image>
-              <width>1280</width>
-              <height>720</height>
-              <format>L_INT8</format>
-            </image>
-            <clip>
-              <near>0.1</near>
-              <far>100</far>
-            </clip>
-            <noise>
-              <type>gaussian</type>
-              <mean>0.0</mean>
-              <stddev>0.05</stddev>
-            </noise>
-          </camera>
-          <always_on>1</always_on>
-          <update_rate>90</update_rate>
-          <visualize>false</visualize>
-          <plugin name="${node_name}_ired2" filename="libgazebo_ros_camera.so">
-            <ros>
-              <namespace>${node_namespace}/${node_name}</namespace>
-            </ros>
-            <camera_name>${node_name}_ired2</camera_name>
-            <frame_name>${frame_prefix}infra2_optical_frame</frame_name>
-          </plugin>
-        </sensor>
-      </gazebo>
-      <gazebo reference="${frame_prefix}depth_frame">
-        <sensor name="${node_namespace}depth" type="depth">
-          <camera name="${frame_prefix}camera">
-            <horizontal_fov>${radians(85.2)}</horizontal_fov>
-            <image>
-              <width>1280</width>
-              <height>720</height>
-            </image>
-            <clip>
-              <near>0.1</near>
-              <far>100</far>
-            </clip>
-            <noise>
-              <type>gaussian</type>
-              <mean>0.0</mean>
-              <stddev>0.100</stddev>
-            </noise>
-          </camera>
-          <always_on>1</always_on>
-          <update_rate>90</update_rate>
-          <visualize>false</visualize>
-          <plugin name="${node_name}_depth" filename="libgazebo_ros_camera.so">
-            <ros>
-              <namespace>${node_namespace}/${node_name}</namespace>
-            </ros>
-            <camera_name>${node_name}_depth</camera_name>
-            <frame_name>${frame_prefix}depth_optical_frame</frame_name>
-          </plugin>
-        </sensor>
-      </gazebo>
-   </xacro:macro>
-   <xacro:macro name="intel_realsense_d435_ignition">
-      <gazebo reference="${frame_prefix}color_frame">
-        <sensor name="${frame_prefix}color" type="camera">
-          <ignition_frame_id>${frame_prefix}link</ignition_frame_id>
-          <camera name="${frame_prefix}camera">
-            <horizontal_fov>${radians(69.4)}</horizontal_fov>
-            <image>
-              <width>1920</width>
-              <height>1080</height>
-              <format>RGB_INT8</format>
-            </image>
-            <clip>
-              <near>0.1</near>
-              <far>100</far>
-            </clip>
-            <noise>
-              <type>gaussian</type>
-              <mean>0.0</mean>
-              <stddev>0.007</stddev>
-            </noise>
-          </camera>
-          <always_on>1</always_on>
-          <update_rate>30</update_rate>
-          <visualize>false</visualize>
-          <topic>/${node_namespace}/${topic_prefix}/color/image_raw</topic>
-        </sensor>
-      </gazebo>
-      <gazebo reference="${frame_prefix}infra1_frame">
-        <sensor name="${frame_prefix}ired1" type="camera">
-          <ignition_frame_id>${frame_prefix}link</ignition_frame_id>
-          <camera name="${frame_prefix}camera">
-            <horizontal_fov>${radians(85.2)}</horizontal_fov>
-            <image>
-              <width>1280</width>
-              <height>720</height>
-              <format>L_INT8</format>
-            </image>
-            <clip>
-              <near>0.1</near>
-              <far>100</far>
-            </clip>
-            <noise>
-              <type>gaussian</type>
-              <mean>0.0</mean>
-              <stddev>0.05</stddev>
-            </noise>
-          </camera>
-          <always_on>1</always_on>
-          <update_rate>90</update_rate>
-          <visualize>false</visualize>
-          <topic>/${node_namespace}/${topic_prefix}/ired1/image_raw</topic>
-        </sensor>
-      </gazebo>
-      <gazebo reference="${frame_prefix}infra2_frame">
-        <sensor name="${frame_prefix}ired2" type="camera">
-          <ignition_frame_id>${frame_prefix}link</ignition_frame_id>
-          <camera name="${frame_prefix}camera">
-            <horizontal_fov>${radians(85.2)}</horizontal_fov>
-            <image>
-              <width>1280</width>
-              <height>720</height>
-              <format>L_INT8</format>
-            </image>
-            <clip>
-              <near>0.1</near>
-              <far>100</far>
-            </clip>
-            <noise>
-              <type>gaussian</type>
-              <mean>0.0</mean>
-              <stddev>0.05</stddev>
-            </noise>
-          </camera>
-          <always_on>1</always_on>
-          <update_rate>90</update_rate>
-          <visualize>false</visualize>
-          <topic>/${node_namespace}/${topic_prefix}/ired2/image_raw</topic>
-        </sensor>
-      </gazebo>
-      <gazebo reference="${frame_prefix}depth_frame">
-        <sensor name="${frame_prefix}depth" type="depth">
-          <ignition_frame_id>${frame_prefix}link</ignition_frame_id>
-          <camera name="${frame_prefix}camera">
-            <horizontal_fov>${radians(85.2)}</horizontal_fov>
-            <image>
-              <width>1280</width>
-              <height>720</height>
-            </image>
-            <clip>
-              <near>0.1</near>
-              <far>100</far>
-            </clip>
-            <noise>
-              <type>gaussian</type>
-              <mean>0.0</mean>
-              <stddev>0.100</stddev>
-            </noise>
-          </camera>
-          <always_on>1</always_on>
-          <update_rate>90</update_rate>
-          <visualize>false</visualize>
-          <topic>/${node_namespace}/${topic_prefix}/depth/image_raw</topic>
-        </sensor>
-      </gazebo>
-      <!-- <gazebo>
-        <plugin name="${node_name}" filename="librealsense_gazebo_plugin.so">
-          <prefix>${node_namespace}</prefix>
-          <depthUpdateRate>60.0</depthUpdateRate>
-          <colorUpdateRate>60.0</colorUpdateRate>
-          <infraredUpdateRate>60.0</infraredUpdateRate>
-          <depthTopicName>${topic_prefix}depth/image_rect_raw</depthTopicName>
-          <depthCameraInfoTopicName>${topic_prefix}depth/camera_info</depthCameraInfoTopicName>
-          <colorTopicName>${topic_prefix}color/image_raw</colorTopicName>
-          <colorCameraInfoTopicName>${topic_prefix}color/camera_info</colorCameraInfoTopicName>
-          <infrared1TopicName>${topic_prefix}infra1/image_raw</infrared1TopicName>
-          <infrared1CameraInfoTopicName>${topic_prefix}infra1/camera_info</infrared1CameraInfoTopicName>
-          <infrared2TopicName>${topic_prefix}infra2/image_raw</infrared2TopicName>
-          <infrared2CameraInfoTopicName>${topic_prefix}infra2/camera_info</infrared2CameraInfoTopicName>
-          <colorOpticalframeName>${frame_prefix}color_optical_frame</colorOpticalframeName>
-          <depthOpticalframeName>${frame_prefix}depth_optical_frame</depthOpticalframeName>
-          <infrared1OpticalframeName>${frame_prefix}infra1_optical_frame</infrared1OpticalframeName>
-          <infrared2OpticalframeName>${frame_prefix}infra2_optical_frame</infrared2OpticalframeName>
-          <rangeMinDepth>0.2</rangeMinDepth>
-          <rangeMaxDepth>10.0</rangeMaxDepth>
-          <pointCloud>true</pointCloud>
-          <pointCloudTopicName>${topic_prefix}depth/color/points</pointCloudTopicName>
-          <pointCloudCutoff>0.5</pointCloudCutoff>
-        </plugin>
-      </gazebo> -->
+      <xacro:camera_plugin
+        node_namespace="${node_namespace}"
+        node_name="${node_name}_color"
+        topic_prefix="${topic_prefix}_color"
+        gazebo_classic="${gazebo_classic}"
+        gazebo_ignition="${gazebo_ignition}"
+        optical_frame="${frame_prefix}color_optical_frame"
+        reference_frame="${frame_prefix}color_frame"
+        horizontal_fov="69.4"
+        vertical_fov="39"
+        video_width="1920"
+        video_height="1080"
+        min_depth="0.1"
+        max_depth="100"
+        rate="30"
+      >
+      </xacro:camera_plugin>
+      <xacro:irred_camera_plugin
+        node_namespace="${node_namespace}"
+        node_name="${node_name}_irred1"
+        topic_prefix="${topic_prefix}_irred1"
+        gazebo_classic="${gazebo_classic}"
+        gazebo_ignition="${gazebo_ignition}"
+        optical_frame="${frame_prefix}infra1_optical_frame"
+        reference_frame="${frame_prefix}infra2_frame"
+        horizontal_fov="85.2"
+        vertical_fov="48"
+        video_width="1280"
+        video_height="720"
+        min_depth="0.1"
+        max_depth="100"
+        rate="30"
+      >
+      </xacro:irred_camera_plugin>
+      <xacro:irred_camera_plugin
+        node_namespace="${node_namespace}"
+        node_name="${node_name}_irred2"
+        topic_prefix="${topic_prefix}_irred2"
+        gazebo_classic="${gazebo_classic}"
+        gazebo_ignition="${gazebo_ignition}"
+        optical_frame="${frame_prefix}infra2_optical_frame"
+        reference_frame="${frame_prefix}infra2_frame"
+        horizontal_fov="85.2"
+        vertical_fov="48"
+        video_width="1280"
+        video_height="720"
+        min_depth="0.1"
+        max_depth="100"
+        rate="30"
+      >
+      </xacro:irred_camera_plugin>
+      <xacro:depth_camera_plugin
+        node_namespace="${node_namespace}"
+        node_name="${node_name}_depth"
+        topic_prefix="${topic_prefix}_depth"
+        gazebo_classic="${gazebo_classic}"
+        gazebo_ignition="${gazebo_ignition}"
+        optical_frame="${frame_prefix}depth_optical_frame"
+        reference_frame="${frame_prefix}depth_frame"
+        horizontal_fov="85.2"
+        vertical_fov="48"
+        video_width="1280"
+        video_height="720"
+        min_depth="0.1"
+        max_depth="100"
+        rate="30"
+      >
+      </xacro:depth_camera_plugin>
   </xacro:macro>
 </robot>

File: Robotnik_ws/src/robotnik_sensors/robotnik_sensors/urdf/imu/vectornav.urdf.xacro (robot description, xacro)
@@ -1,10 +1,11 @@
 <?xml version="1.0"?>
 <robot name="sensor_vectornav" xmlns:xacro="http://wiki.ros.org/xacro">
+  <xacro:include filename="$(find robotnik_sensors)/urdf/imu/imu_plugin.urdf.xacro" />
   <xacro:macro name="sensor_vectornav"
                params="frame_prefix
                        parent
                        *origin
-                       simulation:=false
-                       simulator:=none
+                       gazebo_classic:=false
+                       gazebo_ignition:=false
                        node_name:=imu
                        node_namespace:=${None}
@@ -44,185 +45,16 @@
     </joint>
     <link name="${frame_prefix}link" />
-    <xacro:if value="${simulator == 'gazebo_classic'}">
-      <gazebo reference="${frame_prefix}base_link">
-        <material>Gazebo/Red</material>
-      </gazebo>
-      <gazebo reference="${frame_prefix}link">
-        <gravity>true</gravity>
-        <sensor name="${frame_prefix}sensor" type="imu">
-          <always_on>true</always_on>
-          <update_rate>200</update_rate>
-          <visualize>true</visualize>
-          <imu>
-            <orientation>
-              <x>
-                <noise type="gaussian">
-                  <mean>0.0</mean>
-                  <!-- <stddev>2e-3</stddev> -->
-                  <stddev>0.01</stddev>
-                </noise>
-              </x>
-              <y>
-                <noise type="gaussian">
-                  <mean>0.0</mean>
-                  <!-- <stddev>2e-3</stddev> -->
-                  <stddev>0.01</stddev>
-                </noise>
-              </y>
-              <z>
-                <noise type="gaussian">
-                  <mean>0.0</mean>
-                  <!-- <stddev>2e-3</stddev> -->
-                  <stddev>0.01</stddev>
-                </noise>
-              </z>
-            </orientation>
-            <angular_velocity>
-              <x>
-                <noise type="gaussian">
-                  <mean>0.0</mean>
-                  <!-- <stddev>2e-4</stddev> -->
-                  <stddev>0.01</stddev>
-                </noise>
-              </x>
-              <y>
-                <noise type="gaussian">
-                  <mean>0.0</mean>
-                  <!-- <stddev>2e-4</stddev> -->
-                  <stddev>0.01</stddev>
-                </noise>
-              </y>
-              <z>
-                <noise type="gaussian">
-                  <mean>0.0</mean>
-                  <!-- <stddev>2e-3</stddev> -->
-                  <stddev>0.01</stddev>
-                </noise>
-              </z>
-            </angular_velocity>
-            <linear_acceleration>
-              <x>
-                <noise type="gaussian">
-                  <mean>0.0</mean>
-                  <!-- <stddev>1.7e-2</stddev> -->
-                  <stddev>0.01</stddev>
-                </noise>
-              </x>
-              <y>
-                <noise type="gaussian">
-                  <mean>0.0</mean>
-                  <!-- <stddev>1.7e-2</stddev> -->
-                  <stddev>0.01</stddev>
-                </noise>
-              </y>
-              <z>
-                <noise type="gaussian">
-                  <mean>0.0</mean>
-                  <!-- <stddev>1.7e-2</stddev> -->
-                  <stddev>0.01</stddev>
-                </noise>
-              </z>
-            </linear_acceleration>
-          </imu>
-          <plugin name="${node_name}" filename="libgazebo_ros_imu_sensor.so">
-            <ros>
-              <namespace>${node_namespace}</namespace>
-              <remapping>~/out:=${topic_prefix}data</remapping>
-            </ros>
-            <initial_orientation_as_reference>false</initial_orientation_as_reference>
-            <frame_name>${frame_prefix}link</frame_name>
-          </plugin>
-        </sensor>
-      </gazebo>
-    </xacro:if>
-    <xacro:if value="${simulator == 'gazebo_ignition'}">
-      <gazebo reference="${frame_prefix}base_link">
-        <material>Gazebo/Red</material>
-      </gazebo>
-      <gazebo reference="${frame_prefix}link">
-        <gravity>true</gravity>
-        <sensor name="${frame_prefix}sensor" type="imu">
-          <always_on>true</always_on>
-          <update_rate>200</update_rate>
-          <visualize>true</visualize>
-          <topic>/imu/data</topic>
-          <imu>
-            <orientation>
-              <x>
-                <noise type="gaussian">
-                  <mean>0.0</mean>
-                  <!-- <stddev>2e-3</stddev> -->
-                  <stddev>0.01</stddev>
-                </noise>
-              </x>
-              <y>
-                <noise type="gaussian">
-                  <mean>0.0</mean>
-                  <!-- <stddev>2e-3</stddev> -->
-                  <stddev>0.01</stddev>
-                </noise>
-              </y>
-              <z>
-                <noise type="gaussian">
-                  <mean>0.0</mean>
-                  <!-- <stddev>2e-3</stddev> -->
-                  <stddev>0.01</stddev>
-                </noise>
-              </z>
-            </orientation>
-            <angular_velocity>
-              <x>
-                <noise type="gaussian">
-                  <mean>0.0</mean>
-                  <!-- <stddev>2e-4</stddev> -->
-                  <stddev>0.01</stddev>
-                </noise>
-              </x>
-              <y>
-                <noise type="gaussian">
-                  <mean>0.0</mean>
-                  <!-- <stddev>2e-4</stddev> -->
-                  <stddev>0.01</stddev>
-                </noise>
-              </y>
-              <z>
-                <noise type="gaussian">
-                  <mean>0.0</mean>
-                  <!-- <stddev>2e-3</stddev> -->
-                  <stddev>0.01</stddev>
-                </noise>
-              </z>
-            </angular_velocity>
-            <linear_acceleration>
-              <x>
-                <noise type="gaussian">
-                  <mean>0.0</mean>
-                  <!-- <stddev>1.7e-2</stddev> -->
-                  <stddev>0.01</stddev>
-                </noise>
-              </x>
-              <y>
-                <noise type="gaussian">
-                  <mean>0.0</mean>
-                  <!-- <stddev>1.7e-2</stddev> -->
-                  <stddev>0.01</stddev>
-                </noise>
-              </y>
-              <z>
-                <noise type="gaussian">
-                  <mean>0.0</mean>
-                  <!-- <stddev>1.7e-2</stddev> -->
-                  <stddev>0.01</stddev>
-                </noise>
-              </z>
-            </linear_acceleration>
-          </imu>
-          <plugin name="ignition::gazebo::systems::Imu" filename="libignition-gazebo-imu-system.so">
-            <initial_orientation_as_reference>false</initial_orientation_as_reference>
-            <frame_name>${frame_prefix}link</frame_name>
-          </plugin>
-        </sensor>
-      </gazebo>
-    </xacro:if>
+    <xacro:imu_plugin
+      node_namespace="${node_namespace}"
+      node_name="${node_name}"
+      gazebo_classic="${gazebo_classic}"
+      gazebo_ignition="${gazebo_ignition}"
+      frame_link="${frame_prefix}link"
+      rate="200.0"
+    >
+    </xacro:imu_plugin>
+    <gazebo reference="${frame_prefix}base_link">
+      <material>Gazebo/Red</material>
+    </gazebo>
   </xacro:macro>
 </robot>
