Commit message: Webots controladores (primer intento)

File: Robotnik_ws/src/robot_description/robots/rbrobout/rbrobout.urdf.xacro (robot description, xacro)
@@ -89,6 +89,4 @@
     <xacro:if value="$(arg gazebo_ignition)">
         <xacro:rbrobout_gz_ignition_control namespace="$(arg namespace)" prefix="$(arg prefix)"/>
-        <xacro:ros_diff_move_gazebo_ignition_front prefix="$(arg prefix)"/>
-        <xacro:ros_diff_move_gazebo_ignition_rear prefix="$(arg prefix)"/>
     </xacro:if>
     <xacro:unless value="$(arg gazebo_classic)">

File: Robotnik_ws/src/robot_description/robots/rbwatcher/rbwatcher.urdf.xacro (robot description, xacro)
@@ -94,6 +94,4 @@
 		</xacro:if>
 		<xacro:rbwatcher_gz_ignition_control namespace="$(arg namespace)" prefix="$(arg prefix)"/>
-        	<xacro:ros_diff_move_gazebo_ignition_front prefix="$(arg prefix)"/>
-        	<xacro:ros_diff_move_gazebo_ignition_rear prefix="$(arg prefix)"/>
    </xacro:macro>
    <xacro:rbwatcher prefix="$(arg prefix)" publish_bf="true" hq="true" kinematics="$(arg kinematics)"/>

File: Robotnik_ws/src/robot_description/simulators/gazebo_ignition/rbrobout/rbrobout_control.urdf.xacro (robot description, xacro)
@@ -34,37 +34,3 @@
         </ros2_control>
     </xacro:macro>
-    <xacro:macro name="ros_diff_move_gazebo_ignition_front" params="prefix">
-        <gazebo>
-          <plugin
-             filename="libignition-gazebo-diff-drive-system.so"
-             name="ignition::gazebo::systems::DiffDrive">
-             <left_joint>${prefix}front_left_wheel_joint</left_joint>
-	     <right_joint>${prefix}front_right_wheel_joint</right_joint>
-             <wheel_separation>0.573</wheel_separation>
-             <wheel_radius>0.127</wheel_radius>
-             <odom_publish_frequency>1</odom_publish_frequency>
-             <topic>cmd_vel</topic>
-             <frame_id>robot_odom</frame_id>
-             <child_frame_id>robot_base_footprint</child_frame_id>
-          </plugin>
-        </gazebo>
-    </xacro:macro>
-    <xacro:macro name="ros_diff_move_gazebo_ignition_rear" params="prefix">
-        <gazebo>
-          <plugin
-             filename="libignition-gazebo-diff-drive-system.so"
-             name="ignition::gazebo::systems::DiffDrive">
-	     <left_joint>${prefix}back_left_wheel_joint</left_joint>
-	     <right_joint>${prefix}back_right_wheel_joint</right_joint>
-             <wheel_separation>0.573</wheel_separation>
-             <wheel_radius>0.127</wheel_radius>
-             <odom_publish_frequency>0</odom_publish_frequency>
-             <publish_odom>false</publish_odom>
-             <publish_odom_tf>false</publish_odom_tf>
-             <topic>cmd_vel_rear</topic>
-             <frame_id>robot_odom</frame_id>
-             <child_frame_id>robot_base_footprint</child_frame_id>
-          </plugin>
-        </gazebo>
-    </xacro:macro>
 </robot>

File: Robotnik_ws/src/robot_description/simulators/gazebo_ignition/rbwatcher/rbwatcher_control.urdf.xacro (robot description, xacro)
@@ -35,39 +35,3 @@
         </ros2_control>
     </xacro:macro>
-    <xacro:macro name="ros_diff_move_gazebo_ignition_front" params="prefix">
-        <gazebo>
-          <plugin
-             filename="libignition-gazebo-diff-drive-system.so"
-             name="ignition::gazebo::systems::DiffDrive">
-             <left_joint>${prefix}front_left_wheel_joint</left_joint>
-	     <right_joint>${prefix}front_right_wheel_joint</right_joint>
-             <wheel_separation>0.31</wheel_separation>
-             <wheel_radius>0.11</wheel_radius>
-             <odom_publish_frequency>1</odom_publish_frequency>
-             <topic>cmd_vel</topic>
-             <torque>50</torque>
-             <frame_id>robot_odom</frame_id>
-             <child_frame_id>robot_base_footprint</child_frame_id>
-          </plugin>
-        </gazebo>
-    </xacro:macro>
-    <xacro:macro name="ros_diff_move_gazebo_ignition_rear" params="prefix">
-        <gazebo>
-          <plugin
-             filename="libignition-gazebo-diff-drive-system.so"
-             name="ignition::gazebo::systems::DiffDrive">
-	     <left_joint>${prefix}back_left_wheel_joint</left_joint>
-	     <right_joint>${prefix}back_right_wheel_joint</right_joint>
-             <wheel_separation>0.31</wheel_separation>
-             <wheel_radius>0.11</wheel_radius>
-             <odom_publish_frequency>0</odom_publish_frequency>
-             <publish_odom>false</publish_odom>
-             <publish_odom_tf>false</publish_odom_tf>
-             <topic>cmd_vel_rear</topic>
-             <frame_id>robot_odom</frame_id>
-             <torque>50</torque>
-             <child_frame_id>robot_base_footprint</child_frame_id>
-          </plugin>
-        </gazebo>
-    </xacro:macro>
 </robot>

File: Robotnik_ws/src/robot_description/urdf/wheels/omni_wheel/rbrobout_omni_wheel.urdf.xacro (robot description, xacro)
@@ -18,5 +18,5 @@
       <axis xyz="0 1 0" rpy="0 0 0" />
       <limit effort="100" velocity="100"/>
-      <joint_properties damping="0.5" friction="2.0"/>
+      <joint_properties damping="0.0" friction="0.0"/>
     </joint>
     <link name="${prefix}_wheel_link">
@@ -50,9 +50,9 @@
       </inertial>
     </link>
-    <gazebo reference="${prefix}_wheel_link">
-      <mu1>0.90</mu1>
-      <mu2>0.85</mu2>
-      <kp>2.75e6</kp>
-      <kd>8.25e1</kd>
+    <gazebo reference="${prefix}wheel_link">
+      <mu1>0.0</mu1>
+      <mu2>0.0</mu2>
+      <kp>0</kp>
+      <kd>0</kd>
       <fdir1>0 0 0</fdir1>
     </gazebo>

Commit message: FBX y PROTO de RbTheron y RbVogui

File: Robotnik_ws/src/robot_description/robots/rbrobout/rbrobout.urdf.xacro (robot description, xacro)
@@ -13,5 +13,5 @@
   <xacro:arg name="namespace" default="robot"/>
   <xacro:arg name="prefix" default="robot_"/>
-  <xacro:arg name="gazebo_classic" default="true"/>
+  <xacro:arg name="gazebo_classic" default="false"/>
   <xacro:arg name="gazebo_ignition" default="false"/>
   <xacro:property name="front_laser_offset_x" value="0.8"/>

File: Robotnik_ws/src/robot_description/robots/rbtheron/rbtheron.urdf.xacro (robot description, xacro)
@@ -10,8 +10,7 @@
     <xacro:include filename="$(find robot_description)/urdf/base_hw/rbtheron.ros2_control.urdf" />
 	<xacro:include filename="$(find robot_description)/simulators/gazebo_classic/rbtheron/rbtheron_control.urdf.xacro"/>
+	<xacro:include filename="$(find robot_description)/simulators/gazebo_ignition/rbtheron/rbtheron_control.urdf.xacro"/>
 	<!-- Import all available sensors -->
 	<xacro:include filename="$(find robotnik_sensors)/urdf/all_sensors.urdf.xacro" />
-	<!-- Import Elevator -->
-	<xacro:include filename="$(find robot_description)/urdf/structures/elevator/rb_theron_elevator.urdf.xacro"/>
 	<!-- ***************** -->
 	<!-- Global parameters -->
@@ -21,25 +20,73 @@
 	<!-- Flag to select the high or low quality model -->
 	<xacro:property name="hq" value="true" />
-	<!-- ELEVATOR PARAMETERS -->
-	<xacro:property name="elevator_x" value="0.0" />
-	<xacro:property name="elevator_y" value="0.0" />
-	<xacro:property name="elevator_z" value="0.2238" />
 	<xacro:arg name="namespace" default="robot"/>
 	<xacro:arg name="prefix" default="robot_"/>
-	<xacro:arg name="gazebo_classic" default="false"/>
-    <!-- <xacro:arg name="has_elevator" default="false" /> -->
+	<xacro:arg name="gazebo_classic" default="true"/>
+	<xacro:arg name="gazebo_ignition" default="false"/>
 	<!-- Here we create the robot using the xacro:macro imported at the beggining of this file -->
 	<xacro:rbtheron prefix="$(arg prefix)" hq="${hq}"/>
-  	<!-- PENDIENTE DE ACTUALIZAR ROBOTNIK_SENSORS -->
-	<!-- ELEVATOR_PLATFORM -->
-	<!-- <xacro:if value="$(arg has_elevator)">
-		<xacro:elevator_platform robot_id="rbtheron_elevator" parent="rbtheron_base_link" hq="${hq}">
-			<origin xyz="${elevator_x} -${elevator_y} ${elevator_z}" rpy="1.5708 0 1.5708"/>
-		</xacro:elevator_platform>
-	</xacro:if> -->
 	<!-- SENSORS -->
-	<!-- <xacro:sensor_vectornav prefix="rbtheron_" parent="rbtheron_base_link" topic="imu/data">
-		<origin xyz="-0.1975 0.0 0.1598" rpy="0 0 0"/>
-    </xacro:sensor_vectornav> -->
+    <xacro:property name="imu_offset_x" value="-0.1975"/>
+    <xacro:property name="imu_offset_y" value="0.0"/>
+    <xacro:property name="imu_offset_z" value="0.1598"/>
+	<xacro:property name="front_rgbd_camera_offset_x" value="0.3045"/>
+	<xacro:property name="front_rgbd_camera_offset_y" value="0.0"/>
+	<xacro:property name="front_rgbd_camera_offset_z" value="0.1898"/>
+	<xacro:property name="rear_rgbd_camera_offset_x" value="-0.3045"/>
+	<xacro:property name="rear_rgbd_camera_offset_y" value="0.0"/>
+	<xacro:property name="rear_rgbd_camera_offset_z" value="0.1158"/>
+	<xacro:property name="front_laser_offset_x" value="0.2675"/>
+	<xacro:property name="front_laser_offset_y" value="-0.215"/>
+	<xacro:property name="front_laser_offset_z" value="0.1613"/>
+	<xacro:property name="rear_laser_offset_x" value="-0.2675"/>
+	<xacro:property name="rear_laser_offset_y" value="0.215"/>
+	<xacro:property name="rear_laser_offset_z" value="0.1613"/>
+	<!-- IMU -->
+    <xacro:sensor_vectornav
+        frame_prefix="$(arg prefix)vectornav_"
+        parent="$(arg prefix)base_link"
+        node_namespace="$(arg namespace)"
+        gazebo_classic="$(arg gazebo_classic)"
+        gazebo_ignition="$(arg gazebo_ignition)">
+        <origin xyz="${imu_offset_x} ${imu_offset_y} ${imu_offset_z}" rpy="0 0 0"/>
+    </xacro:sensor_vectornav>
+	<!-- 2D LASER -->
+    <xacro:sensor_hokuyo_ust20lx
+        frame_prefix="$(arg prefix)front_laser_"
+        parent="$(arg prefix)base_link"
+        node_namespace="$(arg namespace)"
+        node_name="front_laser"
+        gazebo_classic="$(arg gazebo_classic)"
+        gazebo_ignition="$(arg gazebo_ignition)">
+        <origin xyz="${front_laser_offset_x} ${front_laser_offset_y} ${front_laser_offset_z}" rpy="0 ${-PI} ${3/4*PI}"/>
+    </xacro:sensor_hokuyo_ust20lx>
+    <xacro:sensor_hokuyo_ust20lx
+        frame_prefix="$(arg prefix)rear_laser_"
+        parent="$(arg prefix)base_link"
+        node_namespace="$(arg namespace)"
+        node_name="rear_laser"
+        gazebo_classic="$(arg gazebo_classic)"
+        gazebo_ignition="$(arg gazebo_ignition)">
+        <origin xyz="${rear_laser_offset_x} ${rear_laser_offset_y} ${rear_laser_offset_z}" rpy="0 ${-PI} ${-1/4*PI}"/>
+    </xacro:sensor_hokuyo_ust20lx>
+  	<!-- CAMERAS -->
+    <xacro:sensor_intel_realsense_d435
+        frame_prefix="$(arg prefix)front_rgbd_camera_"
+        parent="$(arg prefix)base_link"
+        node_namespace="$(arg namespace)"
+        node_name="front_camera"
+        gazebo_classic="$(arg gazebo_classic)"
+        gazebo_ignition="$(arg gazebo_ignition)">
+        <origin xyz="${front_rgbd_camera_offset_x} ${front_rgbd_camera_offset_y} ${front_rgbd_camera_offset_z}" rpy="0 0 0"/>
+    </xacro:sensor_intel_realsense_d435>
+    <xacro:sensor_intel_realsense_d435
+        frame_prefix="$(arg prefix)rear_rgbd_camera_"
+        parent="$(arg prefix)base_link"
+        node_namespace="$(arg namespace)"
+        node_name="rear_camera"
+        gazebo_classic="$(arg gazebo_classic)"
+        gazebo_ignition="$(arg gazebo_ignition)">
+        <origin xyz="${rear_rgbd_camera_offset_x} ${rear_rgbd_camera_offset_y} ${rear_rgbd_camera_offset_z}" rpy="0 0 ${PI}"/>
+    </xacro:sensor_intel_realsense_d435>
 	<!-- Controllers -->
 	<xacro:if value="$(arg gazebo_classic)">
@@ -47,6 +94,11 @@
         <xacro:ros_planar_move_gazebo_classic/>
 	</xacro:if>
-  <xacro:unless value="$(arg gazebo_classic)">
-    <xacro:rbtheron_base_hw_controller/>
-  </xacro:unless>
+	<xacro:if value="$(arg gazebo_ignition)">
+		<xacro:rbtheron_gz_ignition_control namespace="$(arg namespace)" prefix="$(arg prefix)"/>
+	</xacro:if>
+    <xacro:unless value="$(arg gazebo_classic)">
+        <xacro:unless value="$(arg gazebo_ignition)">
+            <xacro:rbtheron_base_hw_controller/>
+        </xacro:unless>
+    </xacro:unless>
 </robot>

File: Robotnik_ws/src/robot_description/robots/rbvogui/rbvogui.urdf.xacro (robot description, xacro)
@@ -37,9 +37,9 @@
     <xacro:arg name="namespace" default="robot" />
     <xacro:arg name="prefix" default="robot_" />
-    <xacro:arg name="gazebo_classic" default="false" />
+    <xacro:arg name="gazebo_classic" default="true" />
     <xacro:arg name="gazebo_ignition" default="false" />
     <xacro:rbvogui prefix="$(arg prefix)" hq="${hq}" />
     <!-- SENSORS see robotnik_sensors for the specific configuration -->
-    <!-- IMU -->
+  <!-- IMU -->
     <xacro:sensor_vectornav
         frame_prefix="$(arg prefix)vectornav_"
@@ -48,5 +48,5 @@
         gazebo_classic="$(arg gazebo_classic)"
         gazebo_ignition="$(arg gazebo_ignition)">
-        <origin xyz="${imu_offset_x} ${imu_offset_y} ${imu_offset_z}" rpy="0 0 0" />
+        <origin xyz="${imu_offset_x} ${imu_offset_y} ${imu_offset_z}" rpy="0 0 0"/>
     </xacro:sensor_vectornav>
     <!-- LASERS -->

File: Robotnik_ws/src/robot_description/urdf/bodies/rbvogui/rbvogui_body.urdf.xacro (robot description, xacro)
@@ -14,5 +14,10 @@
     </joint>
     <!-- BASE_LINK -->
-    <link name="${prefix}base_link"/>
+      <link name="${prefix}base_link">
+          <inertial>
+        <mass value="0.0" />
+        <origin xyz="0 0 0" />
+          </inertial>
+      </link>
     <!-- Chassis -->
     <joint name="${prefix}chassis_joint" type="fixed">

File: Robotnik_ws/src/robotnik_sensors/robotnik_sensors/urdf/2d_lidar/hokuyo_ust20lx.urdf.xacro (robot description, xacro)
@@ -1,9 +1,11 @@
 <?xml version="1.0"?>
 <robot name="sensor_hokuyo_ust20lx" xmlns:xacro="http://wiki.ros.org/xacro">
+  <xacro:include filename="$(find robotnik_sensors)/urdf/2d_lidar/lidar_2d_plugin.urdf.xacro" />
   <xacro:macro name="sensor_hokuyo_ust20lx"
                params="frame_prefix
                        parent
                        *origin
-                       simulation:=false
+                       gazebo_classic:=false
+                       gazebo_ignition:=false
                        node_name:=hokuyo_ust20lx
                        node_namespace:=${None}
@@ -45,44 +47,19 @@
     <link name="${frame_prefix}link"/>
     <!-- Hokuyo sensor for simulation -->
-    <xacro:if value="${simulation}">
-      <xacro:sensor_hokuyo_ust20_gazebo/>
-    </xacro:if>
-  </xacro:macro>
-  <xacro:macro name="sensor_hokuyo_ust20_gazebo">
-    <gazebo reference="${frame_prefix}link">
-			<sensor type="ray" name="${frame_prefix}sensor">
-				<pose>0 0 0 0 0 0</pose>
-				<visualize>false</visualize>
-				<update_rate>40</update_rate>
-				<ray>
-					<scan>
-						<horizontal>
-							<samples>1081</samples>
-							<resolution>1</resolution>
-							<min_angle>-2.3652</min_angle>
-							<max_angle>2.3652</max_angle>
-						</horizontal>
-					</scan>
-					<range>
-						<min>0.06</min>
-						<max>20.0</max>
-						<resolution>0.004359297</resolution>
-					</range>
-					<noise>
-						<type>gaussian</type>
-						<mean>0.0</mean>
-						<stddev>0.01</stddev>
-					</noise>
-				</ray>
-				<plugin name="${node_name}" filename="libgazebo_ros_ray_sensor.so">
-            <ros>
-              <namespace>${node_namespace}</namespace>
-              <remapping>~/out:=~/scan</remapping>
-            </ros>
-            <output_type>sensor_msgs/LaserScan</output_type>
-            <frame_name>${frame_prefix}link</frame_name>
-				</plugin>
-			</sensor>
-	  </gazebo>
+    <xacro:lidar_2d_plugin
+      node_namespace="${node_namespace}"
+      node_name="${node_name}"
+      gazebo_classic="${gazebo_classic}"
+      gazebo_ignition="${gazebo_ignition}"
+      min_range="0.06"
+      max_range="20.0"
+      min_angle="-2.3562"
+      max_angle="2.3562"
+      frame_link="${frame_prefix}link"
+      rate="40"
+      resolution="0.004359297"
+      samples="1081"
+    >
+    </xacro:lidar_2d_plugin>
   </xacro:macro>
 </robot>
